File: hardware/fmcw3.kicad_pcb (KiCad board)
At the start: 4 copper layers, 101.8 x 46.8 mm, 429 parts, among them CON1 SD_Card_DM3BT, CON2 BARREL_JACK, P1 SMA, P10 CONN_01X01, P11 CONN_01X01, P12 CONN_01X01, P13 CONN_01X01, P14 CONN_01X01, P15 CONN_01X01, P16 CONN_01X01, P2 SMA, P3 CONN_02X04, P4 CONN_02X04, P5 CONN_01X01, P6 CONN_01X01, P7 CONN_01X01, P8 CONN_01X01, P9 CONN_01X01, Q1 RE1C002UN, Q2 DNP(RE1C002UN), SW2 SW_PUSH, U1 ADF4158, U10 HMC431LP4, U11 SKY65404, U12 PAT1220-6dB, U13 TRF37A73, U14 MGA-25203, U15 SMA, U16 SKY65404, U17 L7980, U18 L7980, U19 L7980, U2 LP5907-1.8, U20 LP5907-3.0, U21 LP2985A-10DBVR, U22 TPS7A91, U23 TPS7A91, U24 TPS7A91, U25 MIC5301-3.3, U26 5400BL15B050E, U27 5400BL15B050E, U28 5400BL15B050E, U29 ADL5802, U3 PAT1220-6dB, U30 XC7A15T-1FTG256C, U31 USB-MICRO, U32 93LC46B, U33 FT2232H, U34 ADA4940-2, U35 ADA4940-2, U39 LP5907-3.0, U4 KT2520K, U40 W25Q32JV, U5 NC7S04P5X, U6 NB3N551, U7 TLV172DCK, U8 LTC2292, U9 TRF37A73, Y1 ABM10-167-12.000MHZ-T3

Commit message: Current working version.
Parts:
- removed R10: 6.98k, fmcw3:R_0402b
- removed R14: 39k, fmcw3:R_0402b
- removed U14: MGA-25203, fmcw3:MGA-25203
- added C227: 10u, fmcw3:C_0805b, B.Cu at (162.6, 88.9)
- added C228: 100n, fmcw3:C_0402b, B.Cu at (168.9, 86.4)
- added C229: 10n, fmcw3:C_0402b, B.Cu at (166.4, 87.6)
- added C230: 10u, fmcw3:C_0805b, B.Cu at (166.4, 91.4)
- added C231: DNP, fmcw3:C_0805b, B.Cu at (165.1, 85.1)
- added C232: 2.2u, fmcw3:C_0603b, F.Cu at (230.0, 47.1)
- added C233: 100p, fmcw3:C_0402b, F.Cu at (237.6, 40.0)
- added C234: 100p, fmcw3:C_0402b, F.Cu at (220.1, 54.7)
- added FB9: CIC21P101NE, fmcw3:C_0805b, F.Cu at (194.3, 80.0)
- added R19: 6.8k, fmcw3:R_0402b, F.Cu at (165.1, 87.6)
- added R95: 1.47k, fmcw3:R_0402b, F.Cu at (167.6, 86.4)
- added U37: SE2567L, fmcw3:MGA-25203, F.Cu at (214.6, 88.9)
- added U38: TPS7A91, fmcw3:SON-10_2.5x2.5mm, F.Cu at (168.0, 89.9)
- C1, C100, C101, C102, C103, C104, C105, C106, C60, C61, C62, C76, C77, C78, C79, C80, C82, C83, C85, C86, C87, C88, C93, C94, C98: footprint fmcw3:C_0805b -> Capacitor_SMD:C_0805_2012Metric; moved to B.Cu
- C10, C109, C11, C110, C111, C112, C113, C114, C117, C118, C119, C120, C121, C122, C123, C124, C125, C126, C127, C128, C129, C130, C131, C132, C133, C134, C135, C136, C137, C138, C139, C14, C140, C141, C142, C143, C144, C145, C146, C147, C148, C149, C15, C150, C151, C16, C163, C164, C165, C166, C167, C168, C170, C171, C174, C175, C176, C18, C187, C189, C190, C191, C192, C193, C2, C23, C24, C25, C27, C28, C3, C30, C36, C4, C40, C41, C42, C44, C46, C48, C49, C5, C52, C53, C55, C57, C58, C6, C7, C73, C74, C75, C8, C96, C97, C99: footprint fmcw3:C_0402b -> Capacitor_SMD:C_0402_1005Metric
- C107, C162, C26, C38, C64, C70, C71, C72, C81, C84: footprint fmcw3:C_0805b -> Capacitor_SMD:C_0805_2012Metric
- C108, C115, C116, C152, C153, C154, C158, C159, C160, C161, C21, C29, C43: footprint fmcw3:C_0402b -> Capacitor_SMD:C_0402_1005Metric; moved to F.Cu
- C12, C89: footprint fmcw3:C_0603b -> Capacitor_SMD:C_0603_1608Metric; moved to B.Cu
- C13, C17, C63, C65, C66, C67, C68, C69, C9, C90, C91, C92, C95: footprint fmcw3:C_0402b -> Capacitor_SMD:C_0402_1005Metric; moved to B.Cu
- C155, C157, C19, C20, C31: footprint fmcw3:C_0603b -> Capacitor_SMD:C_0603_1608Metric; moved to F.Cu
- C156, C22, C35, C37, C39, C45, C47, C50, C51, C54, C56, C59: footprint fmcw3:C_0603b -> Capacitor_SMD:C_0603_1608Metric
- C169, C210, C216, C217, C218, C222, FB11, FB12, P6, Q2, R1, R104, R111, R112, R114, R115, R118, R20, R21, R3, R38, R41, R43, R44, R45, R46, R47, R48, R49, R5, R50, R6, R69, R7, R70, R73, R79, R8, R82, R83, R87, R89, R90, R94: moved to F.Cu
- C181: footprint Capacitors_SMD:C_1210 -> Capacitor_SMD:C_1210_3225Metric; moved to B.Cu
- C182, C184, C196: footprint Capacitors_SMD:C_1206 -> Capacitor_SMD:C_1206_3216Metric; moved to B.Cu
- C183, C195, C252, R13, R15, R16, R24, R25, R26, R27, R29: moved to B.Cu
- C32: value 100n -> DNP; footprint fmcw3:C_0402b -> Capacitor_SMD:C_0603_1608Metric; moved to F.Cu
- C33: value 100p -> DNP; footprint fmcw3:C_0402b -> Capacitor_SMD:C_0603_1608Metric
- C34: value 100p -> 10u; footprint fmcw3:C_0402b -> Capacitor_SMD:C_0805_2012Metric
- P3, P4: footprint Pin_Headers:Pin_Header_Straight_2x04_Pitch2.54mm_SMD -> Connector_PinHeader_2.54mm:PinHeader_2x04_P2.54mm_Vertical_SMD
- U17, U18, U19: footprint Housings_DFN_QFN:DFN-8-1EP_3x3mm_Pitch0.5mm -> Package_DFN_QFN:DFN-8-1EP_3x3mm_P0.5mm_EP1.66x2.38mm
- U29: footprint Housings_DFN_QFN:QFN-24-1EP_4x4mm_Pitch0.5mm -> Package_DFN_QFN:QFN-24-1EP_4x4mm_P0.5mm_EP2.6x2.6mm
- U33: footprint Housings_QFP:LQFP-64_10x10mm_Pitch0.5mm -> Package_QFP:LQFP-64_10x10mm_P0.5mm
- U40: footprint Housings_DFN_QFN:DFN-S-8-1EP_6x5mm_Pitch1.27mm -> Package_DFN_QFN:DFN-S-8-1EP_6x5mm_P1.27mm
- U5, U7: footprint TO_SOT_Packages_SMD:SOT-353_SC-70-5 -> Package_TO_SOT_SMD:SOT-353_SC-70-5
- U8: footprint Housings_DFN_QFN:QFN-64-1EP_9x9mm_Pitch0.5mm -> Package_DFN_QFN:QFN-64-1EP_9x9mm_P0.5mm_EP4.85x4.85mm
- moved P8 106.4 mm to (222.2, 78.7)
- moved P5 104.1 mm to (114.3, 120.7)
- moved C212 92.1 mm to (184.4, 43.6), turned to 0 degrees
- moved C162 91.4 mm to (116.3, 64.4), turned to 0 degrees
- moved C114 91.2 mm to (118.3, 68.6), turned to 0 degrees
- moved C111 90.9 mm to (119.9, 69.6), turned to 0 degrees
- moved F2 90.6 mm to (121.5, 63.9)
- moved C112 90.4 mm to (119.9, 70.6), turned to 0 degrees
- moved C172 88.5 mm to (129.3, 66.0), turned to 0 degrees
- moved R72 88.4 mm to (180.5, 47.8), turned to 0 degrees
- moved R54 88.4 mm to (121.3, 65.1), turned to 0 degrees
- moved C113 88.3 mm to (122.1, 68.6), turned to 0 degrees
- moved C119 87.7 mm to (119.8, 67.6), turned to 0 degrees
- moved R51 87.5 mm to (117.9, 66.9), turned to 0 degrees
- moved C123 87.0 mm to (123.3, 66.3), turned to 0 degrees
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Connections:
- net /tx/BSW renamed /tx/EN
- C176 pad 1: /1V8 -> /3V3A
- C33 pad 1: Net-(C32-Pad1) -> GND
- C33 pad 2: GND -> Net-(C232-Pad2)
- C34 pad 1: Net-(C32-Pad1) -> GND
- C34 pad 2: GND -> Net-(C232-Pad2)
- R18 pad 1: /1V8 -> /3V3A
Routing:
- net GND: track 555.5 -> 0.00 mm, vias 685 -> 0
- net /3V3D: track 321.3 -> 0.00 mm, vias 49 -> 0
- net /3V3A: track 158.1 -> 0.00 mm, vias 27 -> 0
- net /3V6: track 138.4 -> 0.00 mm, vias 13 -> 0
- net /1V8: track 128.0 -> 0.00 mm, vias 10 -> 0
- net /3V0: track 103.8 -> 0.00 mm, vias 11 -> 0
- net /power/12V: track 93.2 -> 0.00 mm, vias 7 -> 0
- net /1V0: track 89.1 -> 0.00 mm, vias 13 -> 0
- net /fpga/TCK: track 76.7 -> 0.00 mm, vias 6 -> 0
- net /fpga/TDO: track 76.6 -> 0.00 mm, vias 6 -> 0
- net /fpga/PROGRAM_B: track 74.7 -> 0.00 mm, vias 6 -> 0
- net /fpga/TMS: track 74.1 -> 0.00 mm, vias 4 -> 0
- net /fpga/TDI: track 70.8 -> 0.00 mm, vias 6 -> 0
- net /power/5V6: track 64.0 -> 0.00 mm, vias 13 -> 0
- net /fpga/adc/3V0: track 55.1 -> 0.00 mm, vias 7 -> 0
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- removed copper zone on F.Cu, net /1V0
- removed copper zone on In2.Cu, net /1V0
- removed copper zone on B.Cu, net /1V8
- removed copper zone on In2.Cu, net /1V8
- removed copper zone on B.Cu, net /3V0
- removed copper zone on B.Cu, net /3V3A
- removed copper zone on In2.Cu, net /3V3A
- removed copper zone on B.Cu, net /3V3D
- removed copper zone on In2.Cu, net /3V3D
- removed copper zone on B.Cu, net /3V6
- removed copper zone on B.Cu, net /5V
- removed copper zone on B.Cu, net /mixer/5VF
- removed copper zone on B.Cu, net /power/12V
- removed copper zone on F.Cu, net /power/5V6
- removed copper zone on B.Cu, net GND
- removed copper zone on F.Cu, net GND
- removed copper zone on In1.Cu, net GND
- removed copper zone on In2.Cu, net GND
Other:
- board size 101.8 x 46.8 mm -> 123.2 x 49.5 mm
- board text removed: "fmcw3"
