File: hardware/fmcw3.sch (KiCad schematic (older format))
At the start: 20 parts, among them P5 CONN_01X01, P7 CONN_01X01, P8 CONN_01X01, U2 LP5907-1.8, U4 KT2520K, U5 NC7S04P5X, U6 NB3N551

Commit message: Current working version.
Parts:
- C1: footprint fmcw3:C_0805b -> Capacitor_SMD:C_0805_2012Metric; symbol C -> Device:C
- C12: footprint fmcw3:C_0603b -> Capacitor_SMD:C_0603_1608Metric; symbol C -> Device:C
- C13, C15, C16, C17, C9: footprint fmcw3:C_0402b -> Capacitor_SMD:C_0402_1005Metric; symbol C -> Device:C
- FB1: symbol FILTER -> Device:Ferrite_Bead; manf# (none) -> BLM18PG181SH1D
- P5, P7, P8: symbol CONN_01X01 -> fmcw3-rescue:CONN_01X01
- R13, R15, R16, R3, R8: symbol R -> Device:R
- U2: symbol LP5907 -> fmcw3-rescue:LP5907; manf# (none) -> LP5907MFX-1.8/NOPB
- U4: symbol KT2520K -> fmcw3-rescue:KT2520K; manf# (none) -> KT2520K40000DAW18TAS
- U5: footprint TO_SOT_Packages_SMD:SOT-353_SC-70-5 -> Package_TO_SOT_SMD:SOT-353_SC-70-5; symbol 74AHC1G04 -> fmcw3-rescue:74AHC1G04; manf# (none) -> NC7S04P5X
- U6: symbol NB3N551 -> fmcw3-rescue:NB3N551; manf# (none) -> NB3N551MNR4G
Connections:
- net 3V3D: now also FB1.2; no longer FB1.1
- net at C15.1, C17.1, U5.5 (VCC)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: now also FB1.1; no longer FB1.2
Other:
- moved on the sheet: C15, P5, P7, R13, R16
