File: hardware/power.sch (KiCad schematic (older format))
At the start: 96 parts, among them CON2 BARREL_JACK, U17 L7980, U18 L7980, U19 L7980, U20 LP5907-3.0, U21 LP2985A-10DBVR, U22 TPS7A91, U23 TPS7A91, U24 TPS7A91, U25 MIC5301-3.3

Commit message: Current working version.
Parts:
- added C227, C230: 10u, Capacitor_SMD:C_0805_2012Metric, symbol Device:C
- added C228: 100n, Capacitor_SMD:C_0402_1005Metric, symbol Device:C
- added C229: 10n, Capacitor_SMD:C_0402_1005Metric, symbol Device:C
- added C231: DNP, Capacitor_SMD:C_0805_2012Metric, symbol Device:C
- added R19: 6.8k, fmcw3:R_0402b, symbol Device:R
- added R95: 1.47k, fmcw3:R_0402b, symbol Device:R
- added U38: TPS7A91, fmcw3:SON-10_2.5x2.5mm, symbol fmcw3-rescue:TPS7A91
- C100, C101, C102, C103, C104, C105, C106, C169, C172, C177, C178, C60, C61, C62, C64, C70, C71, C72, C76, C77, C78, C79, C80, C81, C82, C83, C84, C85, C86, C87, C88, C93, C94, C98: footprint fmcw3:C_0805b -> Capacitor_SMD:C_0805_2012Metric; symbol C -> Device:C
- C175, C63, C65, C66, C67, C68, C69, C73, C74, C75, C90, C91, C92, C95, C96, C97, C99: footprint fmcw3:C_0402b -> Capacitor_SMD:C_0402_1005Metric; symbol C -> Device:C
- C89: footprint fmcw3:C_0603b -> Capacitor_SMD:C_0603_1608Metric; symbol C -> Device:C
- CON2: symbol BARREL_JACK -> fmcw3-rescue:BARREL_JACK; manf# (none) -> EJ508A
- D1: symbol LED -> Device:LED
- D2, D3: symbol D_Schottky -> fmcw3-rescue:D_Schottky
- D4: symbol D_Schottky -> fmcw3-rescue:D_Schottky; manf# (none) -> SS13FL
- FB11: symbol FILTER -> Device:Ferrite_Bead; manf# (none) -> CIC21P101NE
- L5, L6: symbol INDUCTOR_SMALL -> Device:L
- L7: symbol INDUCTOR_SMALL -> Device:L; manf# (none) -> SRR6040A-330M
- R101, R103, R104, R24, R25, R26, R27, R28, R29, R30, R31, R32, R33, R34, R35, R36, R37, R38, R41, R42, R43, R44, R45, R46, R47, R48: symbol R -> Device:R
- U17, U18, U19: footprint Housings_DFN_QFN:DFN-8-1EP_3x3mm_Pitch0.5mm -> Package_DFN_QFN:DFN-8-1EP_3x3mm_P0.5mm_EP1.66x2.38mm; symbol L7981 -> fmcw3-rescue:L7981; manf# (none) -> L7980TR
- U20: symbol LP5907 -> fmcw3-rescue:LP5907
- U21: symbol LP2985 -> fmcw3-rescue:LP2985
- U22, U23, U24: symbol TPS7A91 -> fmcw3-rescue:TPS7A91; manf# (none) -> TPS7A9101DSKT
- U25: footprint fmcw3:SOT-23-5 -> Package_TO_SOT_SMD:SOT-23-5; symbol MIC5301 -> fmcw3-rescue:MIC5301
Connections:
- net labels added: 4V5
- wire segments 182 -> 294
- no-connect marks 2 -> 3

Commit message: Dropped the 3 from the end of the project name.
Parts:
- CON2: footprint fmcw3:EJ508A -> fmcw:EJ508A; symbol fmcw3-rescue:BARREL_JACK -> fmcw-rescue:BARREL_JACK-fmcw3-rescue
- D1: footprint fmcw3:LED_0603 -> fmcw:LED_0603
- D2, D3, D4: footprint fmcw3:SOD-123F -> fmcw:SOD-123F; symbol fmcw3-rescue:D_Schottky -> fmcw-rescue:D_Schottky-fmcw3-rescue
- FB11: footprint fmcw3:C_0805b -> fmcw:C_0603b
- L5, L6, L7: footprint fmcw3:SRR6040A -> fmcw:SRR6040A
- R101, R103, R104, R19, R24, R25, R26, R27, R28, R29, R30, R31, R32, R33, R34, R35, R36, R37, R38, R41, R42, R43, R44, R45, R46, R47, R48, R95: footprint fmcw3:R_0402b -> fmcw:R_0402b
- U17, U18, U19: symbol fmcw3-rescue:L7981 -> fmcw-rescue:L7981-fmcw3-rescue
- U20: footprint fmcw3:SOT-23-5 -> fmcw:SOT-23-5; symbol fmcw3-rescue:LP5907 -> fmcw-rescue:LP5907-fmcw3-rescue
- U21: footprint fmcw3:SOT-23-5 -> fmcw:SOT-23-5; symbol fmcw3-rescue:LP2985 -> fmcw-rescue:LP2985-fmcw3-rescue
- U22, U23, U24, U38: footprint fmcw3:SON-10_2.5x2.5mm -> fmcw:SON-10_2.5x2.5mm; symbol fmcw3-rescue:TPS7A91 -> fmcw-rescue:TPS7A91-fmcw3-rescue
- U25: symbol fmcw3-rescue:MIC5301 -> fmcw-rescue:MIC5301-fmcw3-rescue
Other:
- moved on the sheet: C100, C101, C102, C103, C104, C105, C230, C231, C67, C68, C69, R19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

Commit message: Modularized LaTeX documentation.
Parts:
- CON2: symbol fmcw-rescue:BARREL_JACK-fmcw3-rescue -> Connector:Barrel_Jack_Switch
Other:
- moved on the sheet: C100, C101, C102, C103, C104, C105, C106, C169, C172, C175, C177, C178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

Commit message: Adjusted power supply for new power amplifier.
Parts:
- removed C169, C231: DNP, Capacitor_SMD:C_0805_2012Metric, symbol Device:C
- removed C227, C230, C60, C61, C79, C80: 10u, Capacitor_SMD:C_0805_2012Metric, symbol Device:C
- removed C228: 100n, Capacitor_SMD:C_0402_1005Metric, symbol Device:C
- removed C229, C63, C65, C66: 10n, Capacitor_SMD:C_0402_1005Metric, symbol Device:C
- removed C67: 39p, Capacitor_SMD:C_0402_1005Metric, symbol Device:C
- removed C68: 100p, Capacitor_SMD:C_0402_1005Metric, symbol Device:C
- removed D2, D3, D4: SS13FL, fmcw:SOD-123F, symbol fmcw-rescue:D_Schottky-fmcw3-rescue
- removed L5, L6: 33u (SRR6040A-330M), fmcw:SRR6040A, symbol Device:L
- removed R101: DNP, fmcw:R_0402b, symbol Device:R
- removed R103: 0, fmcw:R_0402b, symbol Device:R
- removed R32, R34, R36: 4.99k, fmcw:R_0402b, symbol Device:R
- removed R33: 7.5k, fmcw:R_0402b, symbol Device:R
- removed R35: 1k, fmcw:R_0402b, symbol Device:R
- removed R37: 590, fmcw:R_0402b, symbol Device:R
- removed R38: 33, fmcw:R_0402b, symbol Device:R
- removed R41: 56, fmcw:R_0402b, symbol Device:R
- removed R42: 100, fmcw:R_0402b, symbol Device:R
- removed R43: 10.5k, fmcw:R_0402b, symbol Device:R
- removed R44: 2k, fmcw:R_0402b, symbol Device:R
- removed R95: 1.47k, fmcw:R_0402b, symbol Device:R
- removed U17, U18, U19: L7980, Package_DFN_QFN:DFN-8-1EP_3x3mm_P0.5mm_EP1.66x2.38mm, symbol fmcw-rescue:L7981-fmcw3-rescue
- removed U38: TPS7A91, fmcw:SON-10_2.5x2.5mm, symbol fmcw-rescue:TPS7A91-fmcw3-rescue
- added C79, C80: 6TPH100MAEA, symbol Device:CP1
- added D2, D3: SS24FL, symbol Device:D_Schottky
- added L5: SRR1210A-330M, Inductor_SMD:L_Bourns_SRR1210A, symbol Device:L_Core_Ferrite
- added R14: 10k, symbol Device:R
- added U18, U19: TPS5420D, Package_SO:SOIC-8_3.9x4.9mm_P1.27mm, symbol Regulator_Switching:TPS5420D
- added U32: TPS7A7200RGW, Package_DFN_QFN:Texas_VQFN-RGW-20, symbol Regulator_Switching:TPS7A7200RGW
- C100, C103: footprint Capacitor_SMD:C_0805_2012Metric -> (none)
- C69: value 68p -> 10u; footprint Capacitor_SMD:C_0402_1005Metric -> Capacitor_SMD:C_0805_2012Metric
- C73: value 15n -> 10u; footprint Capacitor_SMD:C_0402_1005Metric -> Capacitor_SMD:C_0805_2012Metric
- C74: value 8.2n -> 10u; footprint Capacitor_SMD:C_0402_1005Metric -> Capacitor_SMD:C_0805_2012Metric
- C75: value 4.7n -> 10u; footprint Capacitor_SMD:C_0402_1005Metric -> Capacitor_SMD:C_0805_2012Metric
- C77, C78, C84: value 10u -> 10n; footprint Capacitor_SMD:C_0805_2012Metric -> Capacitor_SMD:C_0402_1005Metric
- C81: value DNP -> 10u
- C82: value 10u -> 10n; footprint Capacitor_SMD:C_0805_2012Metric -> (none)
- C83: value 10u -> 100n; footprint Capacitor_SMD:C_0805_2012Metric -> Capacitor_SMD:C_0402_1005Metric
- C86: value 10u -> DNP; footprint Capacitor_SMD:C_0805_2012Metric -> (none)
- C90: value 100n -> 10u; footprint Capacitor_SMD:C_0402_1005Metric -> Capacitor_SMD:C_0805_2012Metric
- C96: value 10n -> DNP; footprint Capacitor_SMD:C_0402_1005Metric -> Capacitor_SMD:C_0805_2012Metric
- L7: value 33u (SRR6040A-330M) -> SRR1210A-330M; footprint fmcw:SRR6040A -> Inductor_SMD:L_Bourns_SRR1210A; symbol Device:L -> Device:L_Core_Ferrite; manf# SRR6040A-330M -> SRR1210A-330M
- R19: value 6.8k -> 5.11k; footprint fmcw:R_0402b -> (none)
- R25: value 68k -> 10k; footprint fmcw:R_0402b -> (none)
- R26: value 68k -> 2.8k; footprint fmcw:R_0402b -> (none)
- R27: value 15k -> 100k; footprint fmcw:R_0402b -> (none)
- R28: value 59k -> 2.55k
- R29: value 6.8k -> 10.2k
- R30: value 8.2k -> 280k; footprint fmcw:R_0402b -> (none)
- R31: value DNP -> 30.9k; footprint fmcw:R_0402b -> (none)
Connections:
- net labels removed: 4V5, SYNC
- wire segments 294 -> 253
- no-connect marks 3 -> 12
Other:
- moved on the sheet: C101, C104, C106, C172, C175, C177, C178, C62, C64, C70, C71, C72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

Commit message: Documentation for TPS5420D buck converter.
Parts:
- C101, C102, C106, C62, C64, C69, C70, C73, C74, C75, C76, C81, C85, C87, C88, C90, C93, C94, C98: MFN (none) -> 885012107014
- CON2: MFN (none) -> EJ508A; manf# EJ508A -> (none)
- D1: footprint fmcw:LED_0603 -> Diode_SMD:D_0603_1608Metric; MFN (none) -> SML-D12V8WT86
- FB11: value CIC21P101NE -> 74279228600; footprint fmcw:C_0603b -> Capacitor_SMD:C_0603_1608Metric; MFN (none) -> 74279228600; manf# CIC21P101NE -> (none)
- L5, L7: MFN (none) -> SRR1210A-330M; manf# SRR1210A-330M -> (none)
- R24: footprint fmcw:R_0402b -> Resistor_SMD:R_0402_1005Metric; MFN (none) -> ERJ-2RKF2400X
- U18, U19: MFN (none) -> TPS5420D
- U21: footprint fmcw:SOT-23-5 -> fmcw3:SOT-23-5; symbol fmcw-rescue:LP2985-fmcw3-rescue -> Regulator_Linear:LP2985-10.0; MFN (none) -> LP2985A-10DBVR; Spice_Lib_File (none) -> /home/matt/kicad/LP2985-10_PSPICE_TRANS/LP2985-10.LIB; Spice_Model (none) -> LM2985-10; Spice_Netlist_Enabled (none) -> Y; Spice_Primitive (none) -> X
- U22, U23, U24: MFN (none) -> TPS7A9101DSKT; manf# TPS7A9101DSKT -> (none)
Other:
- moved on the sheet: U21
Changed lines of the file:
@@
 F 2 "fmcw:EJ508A" H 3900 2250 60  0001 C CNN
 F 3 "http://www.memoryprotectiondevices.com/datasheets/EJ508A-datasheet.pdf" H 3900 2250 60  0001 C CNN
-F 4 "EJ508A" H 3900 2250 50  0001 C CNN "manf#"
+F 4 "EJ508A" H 3900 2250 50  0001 C CNN "MFN"
 	1    3900 2250
 	1    0    0    -1
@@
 F 2 "Capacitor_SMD:C_0805_2012Metric" H 4788 2250 30  0001 C CNN
 F 3 "" H 4750 2400 60  0000 C CNN
+F 4 "885012107014" H 4750 2400 50  0001 C CNN "MFN"
 	1    4750 2400
 	1    0    0    -1
@@
 P 5200 2150
 F 0 "FB11" V 5150 2000 50  0000 C CNN
-F 1 "CIC21P101NE" V 5050 2100 50  0000 C CNN
-F 2 "fmcw:C_0603b" H 5200 2150 60  0001 C CNN
-F 3 "http://www.samsungsem.com/kr/support/product-search/bead/__icsFiles/afieldfile/2014/11/13/S_CIC21P101NE.pdf" H 5200 2150 60  0001 C CNN
-F 4 "CIC21P101NE" H 5200 2150 50  0001 C CNN "manf#"
+F 1 "74279228600" V 5050 2100 50  0000 C CNN
+F 2 "Capacitor_SMD:C_0603_1608Metric" H 5200 2150 60  0001 C CNN
+F 3 "https://katalog.we-online.de/pbs/datasheet/74279228600.pdf" H 5200 2150 60  0001 C CNN
+F 4 "74279228600" H 5200 2150 50  0001 C CNN "MFN"
 	1    5200 2150
 	0    1    1    0
@@
 F 2 "Capacitor_SMD:C_0805_2012Metric" H 5688 2250 30  0001 C CNN
 F 3 "" H 5650 2400 60  0000 C CNN
+F 4 "885012107014" H 5650 2400 50  0001 C CNN "MFN"
 	1    5650 2400
 	1    0    0    -1
@@
 F 0 "D1" V 2788 2583 50  0000 R CNN
 F 1 "LED" V 2697 2583 50  0000 R CNN
-F 2 "fmcw:LED_0603" H 2750 2700 60  0001 C CNN
+F 2 "Diode_SMD:D_0603_1608Metric" H 2750 2700 60  0001 C CNN
 F 3 "" H 2750 2700 60  0000 C CNN
+F 4 "SML-D12V8WT86" H 2750 2700 50  0001 C CNN "MFN"
 	1    2750 2700
 	0    -1   -1   0
@@
 F 0 "R24" H 2820 2296 50  0000 L CNN
 F 1 "240" H 2820 2205 50  0000 L CNN
-F 2 "fmcw:R_0402b" V 2680 2250 30  0001 C CNN
+F 2 "Resistor_SMD:R_0402_1005Metric" V 2680 2250 30  0001 C CNN
 F 3 "" H 2750 2250 30  0000 C CNN
+F 4 "ERJ-2RKF2400X" H 2750 2250 50  0001 C CNN "MFN"
 	1    2750 2250
 	1    0    0    -1
@@
 F 2 "Capacitor_SMD:C_0805_2012Metric" H 2938 5300 30  0001 C CNN
 F 3 "" H 2900 5450 60  0000 C CNN
+F 4 "885012107014" H 0   0   50  0001 C CNN "MFN"
 	1    2900 5450
 	1    0    0    -1
@@
 F 2 "Inductor_SMD:L_Bourns_SRR1210A" H 5700 5200 60  0001 C CNN
 F 3 "https://www.bourns.com/docs/Product-Datasheets/SRR1210A.pdf" H 5700 5200 60  0001 C CNN
-F 4 "SRR1210A-330M" H 5700 5200 50  0001 C CNN "manf#"
+F 4 "SRR1210A-330M" H 0   0   50  0001 C CNN "MFN"
 	1    5700 5200
 	0    -1   -1   0
@@
 F 2 "Capacitor_SMD:C_0805_2012Metric" H 10288 6700 30  0001 C CNN
 F 3 "" H 10250 6850 60  0000 C CNN
+F 4 "885012107014" H 0   0   50  0001 C CNN "MFN"
 	1    10250 6850
 	1    0    0    -1
@@
 F 2 "Capacitor_SMD:C_0805_2012Metric" H 8888 6500 30  0001 C CNN
 F 3 "" H 8850 6650 60  0000 C CNN
+F 4 "885012107014" H 0   0   50  0001 C CNN "MFN"
 	1    8850 6650
 	1    0    0    -1
@@
 3V0
 $Comp
-L fmcw-rescue:LP2985-fmcw3-rescue U21
+L Regulator_Linear:LP2985-10.0 U21
 U 1 1 596CA417
 P 5100 3650
-F 0 "U21" H 5125 3419 60  0000 C CNN
-F 1 "LP2985A-10DBVR" H 5125 3313 60  0000 C CNN
-F 2 "fmcw:SOT-23-5" H 4850 3450 60  0001 C CNN
-F 3 "" H 4850 3450 60  0001 C CNN
+F 0 "U21" H 5100 3992 50  0000 C CNN
+F 1 "LP2985A-10DBVR" H 5100 3901 50  0000 C CNN
+F 2 "fmcw3:SOT-23-5" H 5100 3975 50  0001 C CNN
+F 3 "http://www.ti.com/lit/ds/symlink/lp2985.pdf" H 5100 3650 50  0001 C CNN
+F 4 "LP2985A-10DBVR" H 5100 3900 50  0001 C CNN "MFN"
+F 5 "/home/matt/kicad/LP2985-10_PSPICE_TRANS/LP2985-10.LIB" H 0   0   50  0001 C CNN "Spice_Lib_File"
+F 6 "LM2985-10" H 0   0   50  0001 C CNN "Spice_Model"
+F 7 "Y" H 0   0   50  0001 C CNN "Spice_Netlist_Enabled"
+F 8 "X" H 0   0   50  0001 C CNN "Spice_Primitive"
 	1    5100 3650
 	1    0    0    -1
@@
 F 2 "Capacitor_SMD:C_0805_2012Metric" H 6188 3600 30  0001 C CNN
 F 3 "" H 6150 3750 60  0000 C CNN
+F 4 "885012107014" H 0   0   50  0001 C CNN "MFN"
 	1    6150 3750
 	1    0    0    -1
@@
 L power:GND #PWR0184
 U 1 1 596CC017
-P 4300 3900
-F 0 "#PWR0184" H 4300 3650 50  0001 C CNN
-F 1 "GND" H 4300 3750 50  0000 C CNN
-F 2 "" H 4300 3900 60  0000 C CNN
-F 3 "" H 4300 3900 60  0000 C CNN
-	1    4300 3900
+P 5100 4050
+F 0 "#PWR0184" H 5100 3800 50  0001 C CNN
+F 1 "GND" H 5100 3900 50  0000 C CNN
+F 2 "" H 5100 4050 60  0000 C CNN
+F 3 "" H 5100 4050 60  0000 C CNN
+	1    5100 4050
 	1    0    0    -1
 $EndComp
@@
 F 2 "fmcw:SON-10_2.5x2.5mm" H 10500 2400 60  0001 C CNN
 F 3 "http://www.ti.com/lit/ds/symlink/tps7a91.pdf" H 10500 2400 60  0001 C CNN
-F 4 "TPS7A9101DSKT" H 10450 2300 50  0001 C CNN "manf#"
+F 4 "" H 10450 2300 50  0001 C CNN "manf#"
+F 5 "TPS7A9101DSKT" H 0   0   50  0001 C CNN "MFN"
 	1    10450 2300
 	1    0    0    -1
@@
 F 2 "Capacitor_SMD:C_0805_2012Metric" H 9088 2000 30  0001 C CNN
 F 3 "" H 9050 2150 60  0000 C CNN
+F 4 "885012107014" H 9050 2150 50  0001 C CNN "MFN"
 	1    9050 2150
 	1    0    0    -1
@@
 F 2 "Capacitor_SMD:C_0805_2012Metric" H 12188 2000 30  0001 C CNN
 F 3 "" H 12150 2150 60  0000 C CNN
+F 4 "885012107014" H 0   0   50  0001 C CNN "MFN"
 	1    12150 2150
 	1    0    0    -1
@@
 F 2 "Capacitor_SMD:C_0805_2012Metric" H 10988 6650 30  0001 C CNN
 F 3 "" H 10950 6800 60  0000 C CNN
+F 4 "885012107014" H 0   0   50  0001 C CNN "MFN"
 	1    10950 6800
 	1    0    0    -1
@@
 F 2 "Capacitor_SMD:C_0805_2012Metric" H 12388 6600 30  0001 C CNN
 F 3 "" H 12350 6750 60  0000 C CNN
+F 4 "885012107014" H 0   0   50  0001 C CNN "MFN"
 	1    12350 6750
 	1    0    0    -1
@@
 F 2 "fmcw:SON-10_2.5x2.5mm" H 10450 5350 60  0001 C CNN
 F 3 "http://www.ti.com/lit/ds/symlink/tps7a91.pdf" H 10450 5350 60  0001 C CNN
-F 4 "TPS7A9101DSKT" H 1600 1550 50  0001 C CNN "manf#"
+F 4 "" H 1600 1550 50  0001 C CNN "manf#"
+F 5 "TPS7A9101DSKT" H 0   0   50  0001 C CNN "MFN"
 	1    10400 5250
 	1    0    0    -1
@@
 F 2 "Capacitor_SMD:C_0805_2012Metric" H 9038 4950 30  0001 C CNN
 F 3 "" H 9000 5100 60  0000 C CNN
+F 4 "885012107014" H 0   0   50  0001 C CNN "MFN"
 	1    9000 5100
 	1    0    0    -1
@@
 F 2 "Capacitor_SMD:C_0805_2012Metric" H 12138 4950 30  0001 C CNN
 F 3 "" H 12100 5100 60  0000 C CNN
+F 4 "885012107014" H 0   0   50  0001 C CNN "MFN"
 	1    12100 5100
 	1    0    0    -1
@@
 Wire Wire Line
 	6150 3600 6150 3550
-Wire Wire Line
-	5700 3550 6150 3550
 Connection ~ 6150 3550
-Wire Wire Line
-	5700 3750 5800 3750
-Wire Wire Line
-	4550 3650 4300 3650
-Wire Wire Line
-	4300 3650 4300 3900
-Wire Wire Line
-	4550 3750 4450 3750
-Wire Wire Line
-	4450 3750 4450 3550
 Connection ~ 4450 3550
 Wire Wire Line
@@
 Wire Wire Line
 	6150 3550 6250 3550
-Wire Wire Line
-	4450 3550 4550 3550
 Wire Wire Line
 	9650 2000 9800 2000
@@
 F 2 "Package_SO:SOIC-8_3.9x4.9mm_P1.27mm" H 4050 5850 50  0001 C CNN
 F 3 "http://www.ti.com/lit/ds/symlink/tps5420.pdf" H 4100 5400 50  0001 C CNN
+F 4 "TPS5420D" H 4100 5400 50  0001 C CNN "MFN"
 	1    4100 5400
 	1    0    0    -1
@@
 F 2 "Capacitor_SMD:C_0805_2012Metric" H 3138 5300 30  0001 C CNN
 F 3 "" H 3100 5450 60  0000 C CNN
+F 4 "885012107014" H 0   0   50  0001 C CNN "MFN"
 	1    3100 5450
 	1    0    0    -1
@@
 F 2 "Capacitor_SMD:C_0805_2012Metric" H 3338 5300 30  0001 C CNN
 F 3 "" H 3300 5450 60  0000 C CNN
+F 4 "885012107014" H 0   0   50  0001 C CNN "MFN"
 	1    3300 5450
 	1    0    0    -1
@@
 F 2 "Capacitor_SMD:C_0805_2012Metric" H 2888 7650 30  0001 C CNN
 F 3 "" H 2850 7800 60  0000 C CNN
+F 4 "885012107014" H 0   0   50  0001 C CNN "MFN"
 	1    2850 7800
 	1    0    0    -1
@@
 F 2 "Package_SO:SOIC-8_3.9x4.9mm_P1.27mm" H 4000 8200 50  0001 C CNN
 F 3 "http://www.ti.com/lit/ds/symlink/tps5420.pdf" H 4050 7750 50  0001 C CNN
+F 4 "TPS5420D" H 0   0   50  0001 C CNN "MFN"
 	1    4050 7750
 	1    0    0    -1
@@
 F 2 "Capacitor_SMD:C_0805_2012Metric" H 3088 7650 30  0001 C CNN
 F 3 "" H 3050 7800 60  0000 C CNN
+F 4 "885012107014" H 0   0   50  0001 C CNN "MFN"
 	1    3050 7800
 	1    0    0    -1
@@
 F 2 "Capacitor_SMD:C_0805_2012Metric" H 3288 7650 30  0001 C CNN
 F 3 "" H 3250 7800 60  0000 C CNN
+F 4 "885012107014" H 0   0   50  0001 C CNN "MFN"
 	1    3250 7800
 	1    0    0    -1
@@
 F 2 "fmcw:SON-10_2.5x2.5mm" H 10350 8200 60  0001 C CNN
 F 3 "http://www.ti.com/lit/ds/symlink/tps7a91.pdf" H 10350 8200 60  0001 C CNN
-F 4 "TPS7A9101DSKT" H 10300 8100 50  0001 C CNN "manf#"
+F 4 "" H 10300 8100 50  0001 C CNN "manf#"
+F 5 "TPS7A9101DSKT" H 0   0   50  0001 C CNN "MFN"
 	1    10300 8100
 	1    0    0    -1
@@
 F 2 "Capacitor_SMD:C_0805_2012Metric" H 8938 7800 30  0001 C CNN
 F 3 "" H 8900 7950 60  0000 C CNN
+F 4 "885012107014" H 0   0   50  0001 C CNN "MFN"
 	1    8900 7950
 	1    0    0    -1
@@
 F 2 "Capacitor_SMD:C_0805_2012Metric" H 12038 7800 30  0001 C CNN
 F 3 "" H 12000 7950 60  0000 C CNN
+F 4 "885012107014" H 0   0   50  0001 C CNN "MFN"
 	1    12000 7950
 	1    0    0    -1
@@
 F 2 "Inductor_SMD:L_Bourns_SRR1210A" H 5650 7550 60  0001 C CNN
 F 3 "https://www.bourns.com/docs/Product-Datasheets/SRR1210A.pdf" H 5650 7550 60  0001 C CNN
-F 4 "SRR1210A-330M" H 5650 7550 50  0001 C CNN "manf#"
+F 4 "SRR1210A-330M" H 0   0   50  0001 C CNN "MFN"
 	1    5650 7550
 	0    -1   -1   0
 $EndComp
+Wire Wire Line
+	4450 3550 4700 3550
+Wire Wire Line
+	5100 4050 5100 3950
+Wire Wire Line
+	4700 3650 4450 3650
+Wire Wire Line
+	4450 3650 4450 3550
+Wire Wire Line
+	5500 3550 6150 3550
+Wire Wire Line
+	5500 3650 5800 3650
+Wire Wire Line
+	5800 3650 5800 3750
 $EndSCHEMATC

Commit message: Made some modifications to the power hardware.
Parts:
- removed C100: 10u, symbol Device:C
- removed C103, C86: DNP, symbol Device:C
- removed C81, C90: 10u, Capacitor_SMD:C_0805_2012Metric, symbol Device:C
- removed C82: 10n, symbol Device:C
- removed C83: 100n, Capacitor_SMD:C_0402_1005Metric, symbol Device:C
- removed C84: 10n, Capacitor_SMD:C_0402_1005Metric, symbol Device:C
- removed C96: DNP, Capacitor_SMD:C_0805_2012Metric, symbol Device:C
- removed R27: 100k, symbol Device:R
- removed R28: 2.55k, fmcw:R_0402b, symbol Device:R
- removed R29: 10.2k, fmcw:R_0402b, symbol Device:R
- removed R30: 280k, symbol Device:R
- removed R31: 30.9k, symbol Device:R
- removed U22: TPS7A91, fmcw:SON-10_2.5x2.5mm, symbol fmcw-rescue:TPS7A91-fmcw3-rescue
- removed U32: TPS7A7200RGW, Package_DFN_QFN:Texas_VQFN-RGW-20, symbol Regulator_Switching:TPS7A7200RGW
- added C? (x7): 10u, Capacitor_SMD:C_0805_2012Metric, symbol Device:C
- added C?: DNP, Capacitor_SMD:C_0805_2012Metric, symbol Device:C
- added C?: 100n, Capacitor_SMD:C_0805_2012Metric, symbol Device:C
- added L?: 10u, symbol Device:L_Core_Ferrite
- added R?: 274k, fmcw:R_0402b, symbol Device:R
- added R?: 30.1k, fmcw:R_0402b, symbol Device:R
- added R?: 4.99k, symbol Device:R
- added R?: 20k, symbol Device:R
- added U?: TPS560200, Package_TO_SOT_SMD:SOT-23-5, symbol Regulator_Switching:TPS560200
- added U?: TPS7A7001DDA, Package_SO:TI_SO-PowerPAD-8, symbol Regulator_Linear:TPS7A7001DDA
- C62, C64, C69, C70, C73, C74, C75, C76, C98: MFN 885012107014 -> GRM21BR61E106MA73L
- C77, C78, C97, C99: MFN (none) -> GRM155R71E103KA01D
- C89: MFN (none) -> CL10A105KA8NNNC
- L5, L7: value SRR1210A-330M -> 33u
- U20: footprint fmcw:SOT-23-5 -> Package_TO_SOT_SMD:SOT-23-5; MFN (none) -> LP5907MFX-3.0/NOPB
Connections:
- wire segments 253 -> 244
- no-connect marks 12 -> 4
Other:
- moved on the sheet: C102, C105, C172, C62, C69, C73, C74, C75, C76, C77, C78, C79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
