File: hardware/power.sch (KiCad schematic (older format))
At the start: 77 parts, among them CON1 BARREL_JACK, U26 TPS5420D, U27 TPS5420D, U28 TPS560200, U29 LP2985A-10DBVR, U30 TPS7A7001DDA, U31 TPS7A91, U32 TPS7A91, U33 LP5907MFX-3.0, U34 TPS7A91

Commit message: Finish FPGA code.
Parts:
- C169, C170, C171, C172, C173, C174, C175, C178, C181, C182, C183, C187, C194, C195, C196, C199, C200, C201, C206, C207, C210, C213: MFN CL21B106KQQNNNE -> ‎CL21B106KOQNNNE‎
Changed lines of the file:
@@
 F 2 "Capacitor_SMD:C_0805_2012Metric" H 4788 2250 30  0001 C CNN
 F 3 "" H 4750 2400 60  0000 C CNN
-F 4 "CL21B106KQQNNNE" H 4750 2400 50  0001 C CNN "MFN"
+F 4 "‎CL21B106KOQNNNE‎" H 4750 2400 50  0001 C CNN "MFN"
 	1    4750 2400
 	1    0    0    -1
@@
 F 2 "Capacitor_SMD:C_0805_2012Metric" H 5688 2250 30  0001 C CNN
 F 3 "" H 5650 2400 60  0000 C CNN
-F 4 "CL21B106KQQNNNE" H 5650 2400 50  0001 C CNN "MFN"
+F 4 "‎CL21B106KOQNNNE‎" H 5650 2400 50  0001 C CNN "MFN"
 	1    5650 2400
 	1    0    0    -1
@@
 F 2 "Capacitor_SMD:C_0805_2012Metric" H 2488 4850 30  0001 C CNN
 F 3 "" H 2450 5000 60  0000 C CNN
-F 4 "CL21B106KQQNNNE" H -450 -450 50  0001 C CNN "MFN"
+F 4 "‎CL21B106KOQNNNE‎" H -450 -450 50  0001 C CNN "MFN"
 	1    2450 5000
 	1    0    0    -1
@@
 F 2 "Capacitor_SMD:C_0805_2012Metric" H 11088 8000 30  0001 C CNN
 F 3 "" H 11050 8150 60  0000 C CNN
-F 4 "CL21B106KQQNNNE" H 800 1300 50  0001 C CNN "MFN"
+F 4 "‎CL21B106KOQNNNE‎" H 800 1300 50  0001 C CNN "MFN"
 	1    11050 8150
 	1    0    0    -1
@@
 F 2 "Capacitor_SMD:C_0805_2012Metric" H 10088 8000 30  0001 C CNN
 F 3 "" H 10050 8150 60  0000 C CNN
-F 4 "CL21B106KQQNNNE" H 1200 1500 50  0001 C CNN "MFN"
+F 4 "‎CL21B106KOQNNNE‎" H 1200 1500 50  0001 C CNN "MFN"
 	1    10050 8150
 	1    0    0    -1
@@
 F 2 "Capacitor_SMD:C_0805_2012Metric" H 6188 3600 30  0001 C CNN
 F 3 "" H 6150 3750 60  0000 C CNN
-F 4 "CL21B106KQQNNNE" H 0   0   50  0001 C CNN "MFN"
+F 4 "‎CL21B106KOQNNNE‎" H 0   0   50  0001 C CNN "MFN"
 	1    6150 3750
 	1    0    0    -1
@@
 F 2 "Capacitor_SMD:C_0805_2012Metric" H 9088 2000 30  0001 C CNN
 F 3 "" H 9050 2150 60  0000 C CNN
-F 4 "CL21B106KQQNNNE" H 9050 2150 50  0001 C CNN "MFN"
+F 4 "‎CL21B106KOQNNNE‎" H 9050 2150 50  0001 C CNN "MFN"
 	1    9050 2150
 	1    0    0    -1
@@
 F 2 "Capacitor_SMD:C_0805_2012Metric" H 12738 2100 30  0001 C CNN
 F 3 "" H 12700 2250 60  0000 C CNN
-F 4 "CL21B106KQQNNNE" H 550 100 50  0001 C CNN "MFN"
+F 4 "‎CL21B106KOQNNNE‎" H 550 100 50  0001 C CNN "MFN"
 	1    12700 2250
 	1    0    0    -1
@@
 F 2 "Capacitor_SMD:C_0805_2012Metric" H 9038 4950 30  0001 C CNN
 F 3 "" H 9000 5100 60  0000 C CNN
-F 4 "CL21B106KQQNNNE" H 0   0   50  0001 C CNN "MFN"
+F 4 "‎CL21B106KOQNNNE‎" H 0   0   50  0001 C CNN "MFN"
 	1    9000 5100
 	1    0    0    -1
@@
 F 2 "Capacitor_SMD:C_0805_2012Metric" H 12288 5050 30  0001 C CNN
 F 3 "" H 12250 5200 60  0000 C CNN
-F 4 "CL21B106KQQNNNE" H 150 100 50  0001 C CNN "MFN"
+F 4 "‎CL21B106KOQNNNE‎" H 150 100 50  0001 C CNN "MFN"
 	1    12250 5200
 	1    0    0    -1
@@
 F 2 "Capacitor_SMD:C_0805_2012Metric" H 2938 4850 30  0001 C CNN
 F 3 "" H 2900 5000 60  0000 C CNN
-F 4 "CL21B106KQQNNNE" H -200 -450 50  0001 C CNN "MFN"
+F 4 "‎CL21B106KOQNNNE‎" H -200 -450 50  0001 C CNN "MFN"
 	1    2900 5000
 	1    0    0    -1
@@
 F 2 "Capacitor_SMD:C_0805_2012Metric" H 3338 4850 30  0001 C CNN
 F 3 "" H 3300 5000 60  0000 C CNN
-F 4 "CL21B106KQQNNNE" H 0   -450 50  0001 C CNN "MFN"
+F 4 "‎CL21B106KOQNNNE‎" H 0   -450 50  0001 C CNN "MFN"
 	1    3300 5000
 	1    0    0    -1
@@
 F 2 "Capacitor_SMD:C_0805_2012Metric" H 2488 6250 30  0001 C CNN
 F 3 "" H 2450 6400 60  0000 C CNN
-F 4 "CL21B106KQQNNNE" H -400 -1400 50  0001 C CNN "MFN"
+F 4 "‎CL21B106KOQNNNE‎" H -400 -1400 50  0001 C CNN "MFN"
 	1    2450 6400
 	1    0    0    -1
@@
 F 2 "Capacitor_SMD:C_0805_2012Metric" H 2938 6250 30  0001 C CNN
 F 3 "" H 2900 6400 60  0000 C CNN
-F 4 "CL21B106KQQNNNE" H -150 -1400 50  0001 C CNN "MFN"
+F 4 "‎CL21B106KOQNNNE‎" H -150 -1400 50  0001 C CNN "MFN"
 	1    2900 6400
 	1    0    0    -1
@@
 F 2 "Capacitor_SMD:C_0805_2012Metric" H 3338 6250 30  0001 C CNN
 F 3 "" H 3300 6400 60  0000 C CNN
-F 4 "CL21B106KQQNNNE" H 50  -1400 50  0001 C CNN "MFN"
+F 4 "‎CL21B106KOQNNNE‎" H 50  -1400 50  0001 C CNN "MFN"
 	1    3300 6400
 	1    0    0    -1
@@
 F 2 "Capacitor_SMD:C_0805_2012Metric" H 2888 7950 30  0001 C CNN
 F 3 "" H 2850 8100 60  0000 C CNN
-F 4 "CL21B106KQQNNNE" H 0   300 50  0001 C CNN "MFN"
+F 4 "‎CL21B106KOQNNNE‎" H 0   300 50  0001 C CNN "MFN"
 	1    2850 8100
 	1    0    0    -1
@@
 F 2 "Capacitor_SMD:C_0805_2012Metric" H 5488 7950 30  0001 C CNN
 F 3 "" H 5450 8100 60  0000 C CNN
-F 4 "CL21B106KQQNNNE" H 2600 300 50  0001 C CNN "MFN"
+F 4 "‎CL21B106KOQNNNE‎" H 2600 300 50  0001 C CNN "MFN"
 	1    5450 8100
 	1    0    0    -1
@@
 F 2 "Capacitor_SMD:C_0805_2012Metric" H 9438 3650 30  0001 C CNN
 F 3 "" H 9400 3800 60  0000 C CNN
-F 4 "CL21B106KQQNNNE" H 9400 3800 50  0001 C CNN "MFN"
+F 4 "‎CL21B106KOQNNNE‎" H 9400 3800 50  0001 C CNN "MFN"
 	1    9400 3800
 	1    0    0    -1
@@
 F 2 "Capacitor_SMD:C_0805_2012Metric" H 12238 3650 30  0001 C CNN
 F 3 "" H 12200 3800 60  0000 C CNN
-F 4 "CL21B106KQQNNNE" H 12200 3800 50  0001 C CNN "MFN"
+F 4 "‎CL21B106KOQNNNE‎" H 12200 3800 50  0001 C CNN "MFN"
 	1    12200 3800
 	1    0    0    -1
@@
 F 2 "Capacitor_SMD:C_0805_2012Metric" H 10588 6350 30  0001 C CNN
 F 3 "" H 10550 6500 60  0000 C CNN
-F 4 "CL21B106KQQNNNE" H 10550 6500 50  0001 C CNN "MFN"
+F 4 "‎CL21B106KOQNNNE‎" H 10550 6500 50  0001 C CNN "MFN"
 	1    10550 6500
 	1    0    0    -1
@@
 F 2 "Capacitor_SMD:C_0805_2012Metric" H 13988 6450 30  0001 C CNN
 F 3 "" H 13950 6600 60  0000 C CNN
-F 4 "CL21B106KQQNNNE" H 1800 4450 50  0001 C CNN "MFN"
+F 4 "‎CL21B106KOQNNNE‎" H 1800 4450 50  0001 C CNN "MFN"
 	1    13950 6600
 	1    0    0    -1
@@
 F 2 "Capacitor_SMD:C_0805_2012Metric" H 5688 7950 30  0001 C CNN
 F 3 "" H 5650 8100 60  0000 C CNN
-F 4 "CL21B106KQQNNNE" H 2800 300 50  0001 C CNN "MFN"
+F 4 "‎CL21B106KOQNNNE‎" H 2800 300 50  0001 C CNN "MFN"
 	1    5650 8100
 	1    0    0    -1
