File: hardware/if.sch (KiCad schematic (older format))
At the start: 30 parts, among them U33 ADA4940-2

Commit message: Changed components to official libs.
Parts:
- added unit 3 of U33
- added unit 4 of U33
- U33: footprint Package_CSP:LFCSP-WQ-24-7EP_4x4mm_P0.5mm_EP2.6416x2.6416mm -> Package_CSP:LFCSP-24-1EP_4x4mm_P0.5mm_EP2.5x2.5mm; symbol fmcw-rescue:ADA4940-2-Amplifier_Difference -> Amplifier_Difference:ADA4940-2; MFN (none) -> ADA4940-2ACPZ-R2
- U33: footprint Package_CSP:LFCSP-WQ-24-7EP_4x4mm_P0.5mm_EP2.6416x2.6416mm -> Package_CSP:LFCSP-24-1EP_4x4mm_P0.5mm_EP2.5x2.5mm; symbol fmcw-rescue:ADA4940-2-Amplifier_Difference -> Amplifier_Difference:ADA4940-2
Connections:
- net 3V3: now also U33.10 (+VS2), U33.3 (+VS1), U33.4 (+VS1), U33.9 (+VS2); no longer U33.10 (+VS), U33.3 (+VS), U33.4 (+VS), U33.9 (+VS)
- net GND: now also U33.15 (-VS2), U33.16 (-VS2), U33.21 (-VS1), U33.22 (-VS1), U33.25 (EP); no longer U33.15 (-VS), U33.16 (-VS), U33.21 (-VS), U33.22 (-VS), U33.25 (EP)
- net OUT1+: now also U33.18 (+OUT1); no longer U33.12 (+OUT)
- net OUT1-: now also U33.19 (-OUT1); no longer U33.13 (-OUT)
- net OUT2+: now also U33.12 (+OUT2); no longer U33.18 (+OUT)
- net OUT2-: now also U33.13 (-OUT2); no longer U33.19 (-OUT)
- net VOCM1: now also U33.11 (VOCM2); no longer U33.17 (VOCM)
- net VOCM2: now also U33.17 (VOCM1); no longer U33.11 (VOCM)
- net at C137.1, R57.1, R61.1: now also U33.7 (-IN2); no longer U33.1 (-IN)
- net at C137.2, R61.2: now also U33.8 (+FB2); no longer U33.2 (+FB)
- net at C136.1, R62.1: now also U33.5 (-FB2); no longer U33.23 (-FB)
- net at C136.2, R58.1, R62.2: now also U33.6 (+IN2); no longer U33.24 (+IN)
- net at C135.1, R55.1, R59.1: now also U33.1 (-IN1); no longer U33.7 (-IN)
- net at C135.2, R59.2: now also U33.2 (+FB1); no longer U33.8 (+FB)
- net at C134.1, R60.1: now also U33.23 (-FB1); no longer U33.5 (-FB)
- net at C134.2, R56.1, R60.2: now also U33.24 (+IN1); no longer U33.6 (+IN)
Other:
- moved on the sheet: C124, C125, C126, C127, C128, C129, C130, C131, C132, C133, C134, C135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

Commit message: Finished design, began routing.
Parts:
- C238: renamed from C126; MFN CL05B223KP5NNNC -> CL05B222KB5VPNC
- C239: renamed from C127; MFN CL05B223KP5NNNC -> CL05B222KB5VPNC
- U39: renamed from U33; MFN (none) -> ADA4940-2ACPZ-R2
- renumbered C139 to C233, C138 to C234, C173 to C235, C124 to C236, C125 to C237, C128 to C240, C129 to C241, C130 to C242, C131 to C243, C132 to C244, C133 to C245, C134 to C246, C136 to C247, C135 to C248, C137 to C249, R55 to R73, R56 to R74, R57 to R75, R58 to R76, R59 to R77, R60 to R78, R61 to R79, R62 to R80, U33 to U39

Commit message: Fixed transmission line width.
Connections:
- net IF1+: now also C237.2, L11.1; no longer C236.2, L9.1
- net IF1-: now also C237.1, L10.1; no longer C236.1, L8.1
- net IF2+: now also C236.2, L9.1; no longer C237.1, L10.1
- net IF2-: now also C236.1, L8.1; no longer C237.2, L11.1
- net OUT1+: now also U39.13 (-OUT2); no longer U39.18 (+OUT1)
- net OUT1-: now also U39.12 (+OUT2); no longer U39.19 (-OUT1)
- net OUT2+: now also U39.18 (+OUT1); no longer U39.12 (+OUT2)
- net OUT2-: now also U39.19 (-OUT1); no longer U39.13 (-OUT2)
- net VOCM1: now also C244.1, U39.17 (VOCM1); no longer C245.1, U39.11 (VOCM2)
- net VOCM2: now also C245.1, U39.11 (VOCM2); no longer C244.1, U39.17 (VOCM1)
Changed lines of the file:
@@
 	1    0    0    -1
 $EndComp
-Text HLabel 4150 2400 0    60   Input ~ 0
+Text HLabel 4300 4850 0    60   Input ~ 0
 IF1-
-Text HLabel 4150 2800 0    60   Input ~ 0
+Text HLabel 4300 5250 0    60   Input ~ 0
 IF1+
 $Comp
@@
 	1    0    0    -1
 $EndComp
-Text HLabel 4300 5250 0    60   Input ~ 0
+Text HLabel 4150 2400 0    60   Input ~ 0
 IF2-
-Text HLabel 4300 4850 0    60   Input ~ 0
+Text HLabel 4150 2800 0    60   Input ~ 0
 IF2+
 $Comp
@@
 	0    1    1    0
 $EndComp
+Text HLabel 8700 4950 2    60   Output ~ 0
+OUT1-
+Text HLabel 8700 5150 2    60   Output ~ 0
+OUT1+
 Text HLabel 8700 2700 2    60   Output ~ 0
-OUT1-
+OUT2-
 Text HLabel 8700 2500 2    60   Output ~ 0
-OUT1+
-Text HLabel 8700 5150 2    60   Output ~ 0
-OUT2-
-Text HLabel 8700 4950 2    60   Output ~ 0
 OUT2+
 $Comp
@@
 Wire Wire Line
 	7450 5150 6700 5150
-Text HLabel 6550 5150 0    60   Input ~ 0
+Text HLabel 6500 2700 0    60   Input ~ 0
 VOCM1
 Wire Wire Line
@@
 Wire Wire Line
 	7450 2700 6700 2700
-Text HLabel 6500 2700 0    60   Input ~ 0
+Text HLabel 6550 5150 0    60   Input ~ 0
 VOCM2
 Wire Wire Line

Commit message: Better MFNs for RF DC blocking caps.
Connections:
- net IF1a-: now reaches C239.1, C242.2, L10.2
- net IF1a+: now reaches C239.2, C243.2, L11.2
- net IF1b-: now reaches C242.1, R75.2
- net IF1b+: now reaches C243.1, R76.2
- net IF2a-: now reaches C238.1, C240.2, L8.2
- net IF2a+: now reaches C238.2, C241.2, L9.2
- net IF2b-: now reaches C240.1, R73.2
- net IF2b+: now reaches C241.1, R74.2
Other:
- moved on the sheet: R73, R74, R75, R76
Changed lines of the file:
@@
 L Device:R R75
 U 1 1 596690B9
-P 6050 4850
-F 0 "R75" V 5843 4850 50  0000 C CNN
-F 1 "549" V 5934 4850 50  0000 C CNN
-F 2 "Resistor_SMD:R_0402_1005Metric" V 5980 4850 30  0001 C CNN
-F 3 "" H 6050 4850 30  0000 C CNN
-F 4 "ERJ-2RKF5490X" H 3150 3100 50  0001 C CNN "MFN"
-	1    6050 4850
+P 6250 4850
+F 0 "R75" V 6043 4850 50  0000 C CNN
+F 1 "549" V 6134 4850 50  0000 C CNN
+F 2 "Resistor_SMD:R_0402_1005Metric" V 6180 4850 30  0001 C CNN
+F 3 "" H 6250 4850 30  0000 C CNN
+F 4 "ERJ-2RKF5490X" H 3350 3100 50  0001 C CNN "MFN"
+	1    6250 4850
 	0    1    1    0
 $EndComp
@@
 L Device:R R76
 U 1 1 59669103
-P 6050 5250
-F 0 "R76" V 6150 5250 50  0000 C CNN
-F 1 "549" V 6250 5250 50  0000 C CNN
-F 2 "Resistor_SMD:R_0402_1005Metric" V 5980 5250 30  0001 C CNN
-F 3 "" H 6050 5250 30  0000 C CNN
-F 4 "ERJ-2RKF5490X" H 3150 3200 50  0001 C CNN "MFN"
-	1    6050 5250
+P 6250 5250
+F 0 "R76" V 6350 5250 50  0000 C CNN
+F 1 "549" V 6450 5250 50  0000 C CNN
+F 2 "Resistor_SMD:R_0402_1005Metric" V 6180 5250 30  0001 C CNN
+F 3 "" H 6250 5250 30  0000 C CNN
+F 4 "ERJ-2RKF5490X" H 3350 3200 50  0001 C CNN "MFN"
+	1    6250 5250
 	0    1    1    0
 $EndComp
@@
 L Device:R R73
 U 1 1 5966BC8A
-P 5900 2400
-F 0 "R73" V 5693 2400 50  0000 C CNN
-F 1 "549" V 5784 2400 50  0000 C CNN
-F 2 "Resistor_SMD:R_0402_1005Metric" V 5830 2400 30  0001 C CNN
-F 3 "" H 5900 2400 30  0000 C CNN
-F 4 "ERJ-2RKF5490X" H 3200 -2550 50  0001 C CNN "MFN"
-	1    5900 2400
+P 6050 2400
+F 0 "R73" V 5843 2400 50  0000 C CNN
+F 1 "549" V 5934 2400 50  0000 C CNN
+F 2 "Resistor_SMD:R_0402_1005Metric" V 5980 2400 30  0001 C CNN
+F 3 "" H 6050 2400 30  0000 C CNN
+F 4 "ERJ-2RKF5490X" H 3350 -2550 50  0001 C CNN "MFN"
+	1    6050 2400
 	0    1    1    0
 $EndComp
@@
 L Device:R R74
 U 1 1 5966BC90
-P 5900 2800
-F 0 "R74" V 6000 2800 50  0000 C CNN
-F 1 "549" V 6100 2800 50  0000 C CNN
-F 2 "Resistor_SMD:R_0402_1005Metric" V 5830 2800 30  0001 C CNN
-F 3 "" H 5900 2800 30  0000 C CNN
-F 4 "ERJ-2RKF5490X" H 3200 -2450 50  0001 C CNN "MFN"
-	1    5900 2800
+P 6050 2800
+F 0 "R74" V 6150 2800 50  0000 C CNN
+F 1 "549" V 6250 2800 50  0000 C CNN
+F 2 "Resistor_SMD:R_0402_1005Metric" V 5980 2800 30  0001 C CNN
+F 3 "" H 6050 2800 30  0000 C CNN
+F 4 "ERJ-2RKF5490X" H 3350 -2450 50  0001 C CNN "MFN"
+	1    6050 2800
 	0    1    1    0
 $EndComp
@@
 	8000 3950 8000 4050
 Wire Wire Line
-	5900 4850 5800 4850
+	6100 4850 5800 4850
 Connection ~ 7750 6100
 Wire Wire Line
-	5900 5250 5800 5250
+	6100 5250 5800 5250
 Wire Wire Line
 	7300 3950 7750 3950
@@
 	8000 1550 8000 1650
 Wire Wire Line
-	5750 2400 5650 2400
+	5900 2400 5650 2400
 Connection ~ 7750 3550
 Wire Wire Line
-	5750 2800 5650 2800
+	5900 2800 5650 2800
 Connection ~ 2500 1950
 Wire Wire Line
@@
 Connection ~ 7750 2050
 Wire Wire Line
-	6050 2400 7300 2400
+	6200 2400 7300 2400
 Wire Wire Line
 	7300 1550 7300 2400
@@
 	5000 2750 5000 2800
 Wire Wire Line
-	6050 2800 7300 2800
+	6200 2800 7300 2800
 Wire Wire Line
 	7300 3550 7750 3550
@@
 	7300 2800 7450 2800
 Wire Wire Line
-	6200 4850 7300 4850
+	6400 4850 7300 4850
 Wire Wire Line
 	7300 3950 7300 4850
@@
 	5150 5150 5150 5250
 Wire Wire Line
-	6200 5250 7300 5250
+	6400 5250 7300 5250
 Wire Wire Line
 	7300 5250 7300 6100
@@
 	1    0    0    -1
 $EndComp
+Text Label 5150 2400 0    50   ~ 0
+IF2a-
+Text Label 5150 2800 0    50   ~ 0
+IF2a+
+Text Label 5700 2800 0    50   ~ 0
+IF2b+
+Text Label 5700 2400 0    50   ~ 0
+IF2b-
+Text Label 5250 4850 0    50   ~ 0
+IF1a-
+Text Label 5250 5250 0    50   ~ 0
+IF1a+
+Text Label 5850 4850 0    50   ~ 0
+IF1b-
+Text Label 5850 5250 0    50   ~ 0
+IF1b+
 $EndSCHEMATC

Commit message: Replaced relevant footprints for thermal via variety.
Parts:
- U39: footprint Package_CSP:LFCSP-24-1EP_4x4mm_P0.5mm_EP2.5x2.5mm -> Package_CSP:LFCSP-24-1EP_4x4mm_P0.5mm_EP2.5x2.5mm_ThermalVias
Changed lines of the file:
@@
 F 0 "U39" H 8050 2900 50  0000 C CNN
 F 1 "ADA4940-2" H 8150 2800 50  0000 C CNN
-F 2 "Package_CSP:LFCSP-24-1EP_4x4mm_P0.5mm_EP2.5x2.5mm" H 7750 2000 50  0001 C CNN
+F 2 "Package_CSP:LFCSP-24-1EP_4x4mm_P0.5mm_EP2.5x2.5mm_ThermalVias" H 7750 2000 50  0001 C CNN
 F 3 "" H 7450 3050 50  0001 C CNN
 F 4 "ADA4940-2ACPZ-R2" H 7750 2600 50  0001 C CNN "MFN"
@@
 F 0 "U39" H 8050 5350 50  0000 C CNN
 F 1 "ADA4940-2" H 8150 5250 50  0000 C CNN
-F 2 "Package_CSP:LFCSP-24-1EP_4x4mm_P0.5mm_EP2.5x2.5mm" H 7750 4450 50  0001 C CNN
+F 2 "Package_CSP:LFCSP-24-1EP_4x4mm_P0.5mm_EP2.5x2.5mm_ThermalVias" H 7750 4450 50  0001 C CNN
 F 3 "" H 7450 5500 50  0001 C CNN
 F 4 "ADA4940-2ACPZ-R2" H 0   0   50  0001 C CNN "MFN"
@@
 F 0 "U39" H 2652 2896 50  0000 L CNN
 F 1 "ADA4940-2" H 2652 2805 50  0000 L CNN
-F 2 "Package_CSP:LFCSP-24-1EP_4x4mm_P0.5mm_EP2.5x2.5mm" H 2500 2450 50  0001 C CNN
+F 2 "Package_CSP:LFCSP-24-1EP_4x4mm_P0.5mm_EP2.5x2.5mm_ThermalVias" H 2500 2450 50  0001 C CNN
 F 3 "" H 800 4050 50  0001 C CNN
 F 4 "ADA4940-2ACPZ-R2" H 0   0   50  0001 C CNN "MFN"
@@
 F 0 "U39" H 2602 5296 50  0000 L CNN
 F 1 "ADA4940-2" H 2602 5205 50  0000 L CNN
-F 2 "Package_CSP:LFCSP-24-1EP_4x4mm_P0.5mm_EP2.5x2.5mm" H 2550 4850 50  0001 C CNN
+F 2 "Package_CSP:LFCSP-24-1EP_4x4mm_P0.5mm_EP2.5x2.5mm_ThermalVias" H 2550 4850 50  0001 C CNN
 F 3 "" H 850 6450 50  0001 C CNN
 F 4 "ADA4940-2ACPZ-R2" H 0   0   50  0001 C CNN "MFN"
