File: hardware/mixer.sch (KiCad schematic (older format))
At the start: 31 parts, among them U35 5400BL15B050E, U36 5400BL15B050E, U37 5400BL15B050E, U38 ADL5802

Commit message: Completed receivers.
Connections:
- net LOIb+: now reaches C220.1, U38.9 (LOIP)
- net LOIa+: now reaches C220.2, U35.4
- net LOIb-: now reaches C221.1, U38.10 (LOIN)
- net LOIa-: now reaches C221.2, U35.3
Changed lines of the file:
@@
 Text Label 4650 4550 0    50   ~ 0
 RF2b-
+Text Label 3350 4600 0    50   ~ 0
+LOIa+
+Text Label 3350 4200 0    50   ~ 0
+LOIa-
+Text Label 4650 4250 0    50   ~ 0
+LOIb+
+Text Label 4650 4350 0    50   ~ 0
+LOIb-
 $EndSCHEMATC

Commit message: Replaced relevant footprints for thermal via variety.
Parts:
- U38: footprint Package_CSP:LFCSP-24-1EP_4x4mm_P0.5mm_EP2.5x2.5mm -> Package_CSP:LFCSP-24-1EP_4x4mm_P0.5mm_EP2.5x2.5mm_ThermalVias
Changed lines of the file:
@@
 F 0 "U38" H 5300 5100 60  0000 C CNN
 F 1 "ADL5802" H 5850 5100 60  0000 C CNN
-F 2 "Package_CSP:LFCSP-24-1EP_4x4mm_P0.5mm_EP2.5x2.5mm" H 5600 4450 60  0001 C CNN
+F 2 "Package_CSP:LFCSP-24-1EP_4x4mm_P0.5mm_EP2.5x2.5mm_ThermalVias" H 5600 4450 60  0001 C CNN
 F 3 "" H 5600 4450 60  0001 C CNN
 F 4 "ADL5802ACPZ-R7" H 950 300 50  0001 C CNN "MFN"

Commit message: Finish FPGA code.
Parts:
- C228: MFN CL21B106KQQNNNE -> ‎CL21B106KOQNNNE‎
Changed lines of the file:
@@
 F 2 "Capacitor_SMD:C_0805_2012Metric" H 6288 2650 30  0001 C CNN
 F 3 "" H 6250 2800 60  0000 C CNN
-F 4 "CL21B106KQQNNNE" H 0   0   50  0001 C CNN "MFN"
+F 4 "‎CL21B106KOQNNNE‎" H 0   0   50  0001 C CNN "MFN"
 	1    6250 2800
 	-1   0    0    1
