File: hardware/antenna-switch/RF_Switch.sch (KiCad schematic (older format))
At the start: 32 parts, among them J8 Conn_01x04, U40 SN74LVC2G14, U41 HMC7992, U42 HMC7992

Commit message: Huge, messy commit before I begin replacing FPGA code
Parts:
- J8: footprint Connector_PinHeader_1.27mm:PinHeader_1x04_P1.27mm_Vertical -> Connector_PinHeader_2.54mm:PinHeader_1x04_P2.54mm_Vertical
Changed lines of the file:
@@
-EESchema Schematic File Version 4
-EELAYER 26 0
+EESchema Schematic File Version 5
+LIBS:antenna_switch-cache
+EELAYER 30 0
 EELAYER END
 $Descr A4 11693 8268
@@
 Comment3 ""
 Comment4 ""
+Comment5 ""
+Comment6 ""
+Comment7 ""
+Comment8 ""
+Comment9 ""
 $EndDescr
 $Comp
@@
 F 0 "J8" H 6330 5792 50  0000 L CNN
 F 1 "Conn_01x04" H 6330 5701 50  0000 L CNN
-F 2 "Connector_PinHeader_1.27mm:PinHeader_1x04_P1.27mm_Vertical" H 6250 5800 50  0001 C CNN
+F 2 "Connector_PinHeader_2.54mm:PinHeader_1x04_P2.54mm_Vertical" H 6250 5800 50  0001 C CNN
 F 3 "~" H 6250 5800 50  0001 C CNN
 	1    6250 5800
