File: hardware/main-pcb/fmcw.kicad_pcb (KiCad board)
At the start: 4 copper layers, 119.6 x 58.9 mm, 415 parts, among them CON1 BARREL_JACK, J1 SD_Card, J2 USB_B_Micro, J3 SMA, J4 SMA, J5 SMA, P1 CONN_02X04, P2 CONN_02X04, Q1 DNP(RE1C002UN), Q2 RE1C002UN, SW1 SW_PUSH, U1 LP5907MFX-3.3, U10 LP5907MFX-3.0, U11 LTC2292, U12 ADF4158, U13 TLV172DCK, U14 PAT1220-C-3DB, U15 HMC431LP4, U16 PD4859J5050S2HF, U17 PAT1220-C-5DB, U18 SE5004L, U19 DC4759J5020AHF, U2 LP5907MFX-1.8, U20 PAT1220-C-6DB, U21 LMV321, U22 TRF37A73, U23 SKY65404, U24 TRF37A73, U25 SKY65404, U26 TPS5420D, U27 TPS5420D, U28 TPS560200, U29 LP2985A-10DBVR, U3 KT2520K-T, U30 TPS7A7001DDA, U31 TPS7A91, U32 TPS7A91, U33 LP5907MFX-3.0, U34 TPS7A91, U35 5400BL15B050E, U36 5400BL15B050E, U37 5400BL15B050E, U38 ADL5802, U39 ADA4940-2, U4 NC7SVU04P5X, U5 NB3N551, U6 XC7A15T-FTG256, U7 W25Q32JV, U8 93LCxxBxxOT, U9 FT2232H, Y1 12MHz

Commit message: pcb: connect ADC reference to voltage supply rail
Connections:
- C77 pad 1: Net-(C77-Pad1) -> /fpga/adc/3V0
- C84 pad 1: Net-(C77-Pad1) -> /fpga/adc/3V0
- C91 pad 1: Net-(C77-Pad1) -> /fpga/adc/3V0
- C95 pad 1: Net-(C77-Pad1) -> /fpga/adc/3V0
- C98 pad 1: Net-(C77-Pad1) -> /fpga/adc/3V0
- C99 pad 1: Net-(C77-Pad1) -> /fpga/adc/3V0
- U10 pad 5: Net-(C77-Pad1) -> /fpga/adc/3V0
- U11 pad 10: Net-(C77-Pad1) -> /fpga/adc/3V0
- U11 pad 18: Net-(C77-Pad1) -> /fpga/adc/3V0
- U11 pad 63: Net-(C77-Pad1) -> /fpga/adc/3V0
- U11 pad 7: Net-(C77-Pad1) -> /fpga/adc/3V0
Routing:
- net Net-(C77-Pad1): track 36.1 -> 0.00 mm, vias 6 -> 0
- net /fpga/adc/3V0: track 5.50 -> 41.6 mm, vias 5 -> 11
