File: hardware/main-pcb/if.sch (KiCad schematic (older format))
At the start: 30 parts, among them U39 ADA4940-2

Commit message: pcb: connect ADC reference to voltage supply rail
Parts:
- U39: symbol Amplifier_Difference:ADA4940-2 -> fmcw-rescue:ADA4940-2-Amplifier_Difference
Changed lines of the file:
@@
 EESchema Schematic File Version 4
 LIBS:fmcw-cache
-EELAYER 26 0
+EELAYER 30 0
 EELAYER END
 $Descr A4 11693 8268
@@
 3V3
 $Comp
-L Amplifier_Difference:ADA4940-2 U?
+L fmcw-rescue:ADA4940-2-Amplifier_Difference U?
 U 1 1 5C3DAB96
 P 7750 2600
@@
 	7750 5600 7750 5700
 $Comp
-L Amplifier_Difference:ADA4940-2 U?
+L fmcw-rescue:ADA4940-2-Amplifier_Difference U?
 U 2 1 5C5E7E6D
 P 7750 5050
@@
 	7300 5250 7450 5250
 $Comp
-L Amplifier_Difference:ADA4940-2 U39
+L fmcw-rescue:ADA4940-2-Amplifier_Difference U39
 U 3 1 5C404FEA
 P 2500 2850
@@
 $EndComp
 $Comp
-L Amplifier_Difference:ADA4940-2 U39
+L fmcw-rescue:ADA4940-2-Amplifier_Difference U39
 U 4 1 5C40EFFA
 P 2550 5250
