File: hardware/main-pcb/usb.sch (KiCad schematic (older format))
At the start: 37 parts, among them J2 USB_B_Micro, U8 93LCxxBxxOT, U9 FT2232H, Y1 12MHz

Commit message: pcb: connect ADC reference to voltage supply rail
Parts:
- U8: symbol Memory_EEPROM:93LCxxBxxOT -> fmcw-rescue:93LCxxBxxOT-Memory_EEPROM
Changed lines of the file:
@@
 EESchema Schematic File Version 4
 LIBS:fmcw-cache
-EELAYER 26 0
+EELAYER 30 0
 EELAYER END
 $Descr A4 11693 8268
@@
 3V3D
 $Comp
-L Memory_EEPROM:93LCxxBxxOT U8
+L fmcw-rescue:93LCxxBxxOT-Memory_EEPROM U8
 U 1 1 5C920D7F
 P 3500 7050
