File: hardware/boards/rev2/adc.sch (KiCad schematic (older format))
At the start: 36 parts, among them U10 LP5907MFX-3.0, U11 LTC2292

Commit message: reorganize schematic
Other:
- note added: "3 mA"
- note added: "95 (78) mA"

Commit message: revert to kicad v5 for pcb gen
V6 contains a few bugs and a V6 board cannot be edited with V5.
Connections:
- net OVDD renamed 3V3D
Changed lines of the file:
@@
-EESchema Schematic File Version 5
-EELAYER 33 0
+EESchema Schematic File Version 4
+EELAYER 30 0
 EELAYER END
 $Descr A4 11693 8268
 encoding utf-8
-Sheet 11 11
+Sheet 3 11
 Title "FMCW"
 Date ""
@@
 Comment3 ""
 Comment4 ""
-Comment5 ""
-Comment6 ""
-Comment7 ""
-Comment8 ""
-Comment9 ""
 $EndDescr
 Connection ~ 7300 6200
@@
 SHDNB
 Text HLabel 8400 1650 2    60   Input ~ 0
-OVDD
+3V3D
 $Comp
 L power:GND #PWR069
