File: hardware/boards/rev2/clock.sch (KiCad schematic (older format))
At the start: 21 parts, among them U1 LP5907MFX-3.3, U2 LP5907MFX-1.8, U3 KT2520K-T, U4 NC7SVU04P5X, U5 NB3N551

Commit message: revert to kicad v5 for pcb gen
V6 contains a few bugs and a V6 board cannot be edited with V5.
Connections:
- net ADC_REF: now also R5.1; no longer R81.1
- net ADF_REF: now also R81.1; no longer R4.1
- net FPGA_REF: now also R4.1; no longer R5.1
Changed lines of the file:
@@
-EESchema Schematic File Version 5
-EELAYER 33 0
+EESchema Schematic File Version 4
+EELAYER 30 0
 EELAYER END
 $Descr A4 11693 8268
 encoding utf-8
-Sheet 11 11
+Sheet 2 11
 Title ""
 Date ""
@@
 Comment3 ""
 Comment4 ""
-Comment5 ""
-Comment6 ""
-Comment7 ""
-Comment8 ""
-Comment9 ""
 $EndDescr
 Connection ~ 5800 2050
@@
 3V6
 Text HLabel 9700 4150 2    50   Output Italic 0
+FPGA_REF
+Text HLabel 9700 4400 2    50   Output Italic 0
 ADF_REF
-Text HLabel 9700 4400 2    50   Output Italic 0
+Text HLabel 9700 4650 2    50   Output Italic 0
 ADC_REF
-Text HLabel 9700 4650 2    50   Output Italic 0
-FPGA_REF
 $Comp
 L power:PWR_FLAG #FLG0101

Commit message: finish placement and routing
Connections:
- net ADC_REF: now also R81.1; no longer R5.1
- net ADF_REF: now also R4.1; no longer R81.1
- net FPGA_REF: now also R5.1; no longer R4.1
Other:
- moved on the sheet: R4, R5, R81
Changed lines of the file:
@@
 	9100 3800 9100 3750
 Wire Wire Line
-	9100 4300 9250 4300
-Wire Wire Line
-	9100 4400 9250 4400
-Wire Wire Line
-	9100 4500 9250 4500
-Wire Wire Line
-	9550 4300 9600 4300
-Wire Wire Line
-	9550 4400 9700 4400
-Wire Wire Line
-	9550 4500 9600 4500
-Wire Wire Line
-	9600 4150 9700 4150
-Wire Wire Line
-	9600 4300 9600 4150
-Wire Wire Line
-	9600 4500 9600 4650
-Wire Wire Line
-	9600 4650 9700 4650
+	9500 4150 9650 4150
+Wire Wire Line
+	9500 4650 9650 4650
+Wire Wire Line
+	9950 4400 10100 4400
 Text Notes 2250 4200 0    59   Italic 0
 2 mA
@@
 Text HLabel 5600 2050 0    50   Input Italic 0
 3V6
-Text HLabel 9700 4150 2    50   Output Italic 0
+Text HLabel 10100 4650 2    50   Output Italic 0
 FPGA_REF
-Text HLabel 9700 4400 2    50   Output Italic 0
+Text HLabel 10100 4150 2    50   Output Italic 0
 ADF_REF
-Text HLabel 9700 4650 2    50   Output Italic 0
+Text HLabel 10100 4400 2    50   Output Italic 0
 ADC_REF
 $Comp
@@
 L Device:R R4
 U 1 1 59741D92
-P 9400 4300
-F 0 "R4" V 9193 4300 50  0000 C CNN
-F 1 "33" V 9284 4300 50  0000 C CNN
-F 2 "Resistor_SMD:R_0402_1005Metric" V 9330 4300 30  0001 C CNN
-F 3 "" H 9400 4300 30  0000 C CNN
-F 4 "" H 3450 -2200 50  0001 C CNN "MFN"
-	1    9400 4300
+P 9800 4150
+F 0 "R4" V 9593 4150 50  0000 C CNN
+F 1 "33" V 9684 4150 50  0000 C CNN
+F 2 "Resistor_SMD:R_0402_1005Metric" V 9730 4150 30  0001 C CNN
+F 3 "" H 9800 4150 30  0000 C CNN
+F 4 "" H 3850 -2350 50  0001 C CNN "MFN"
+	1    9800 4150
 	0    1    1    0
 $EndComp
@@
 L Device:R R81
 U 1 1 5C461FC3
-P 9400 4400
-F 0 "R81" V 9350 4600 50  0000 C CNN
-F 1 "33" V 9400 4400 50  0000 C CNN
-F 2 "Resistor_SMD:R_0402_1005Metric" V 9330 4400 30  0001 C CNN
-F 3 "" H 9400 4400 30  0000 C CNN
-F 4 "" H 3450 -2600 50  0001 C CNN "MFN"
-	1    9400 4400
+P 9800 4400
+F 0 "R81" V 9700 4400 50  0000 C CNN
+F 1 "33" V 9900 4400 50  0000 C CNN
+F 2 "Resistor_SMD:R_0402_1005Metric" V 9730 4400 30  0001 C CNN
+F 3 "" H 9800 4400 30  0000 C CNN
+F 4 "" H 3850 -2600 50  0001 C CNN "MFN"
+	1    9800 4400
 	0    1    1    0
 $EndComp
@@
 L Device:R R5
 U 1 1 5974223B
-P 9400 4500
-F 0 "R5" V 9515 4500 50  0000 C CNN
-F 1 "33" V 9606 4500 50  0000 C CNN
-F 2 "Resistor_SMD:R_0402_1005Metric" V 9330 4500 30  0001 C CNN
-F 3 "" H 9400 4500 30  0000 C CNN
-F 4 "" H 3450 -2500 50  0001 C CNN "MFN"
-	1    9400 4500
+P 9800 4650
+F 0 "R5" V 9915 4650 50  0000 C CNN
+F 1 "33" V 10006 4650 50  0000 C CNN
+F 2 "Resistor_SMD:R_0402_1005Metric" V 9730 4650 30  0001 C CNN
+F 3 "" H 9800 4650 30  0000 C CNN
+F 4 "" H 3850 -2350 50  0001 C CNN "MFN"
+	1    9800 4650
 	0    1    1    0
 $EndComp
@@
 	1    0    0    -1
 $EndComp
+Wire Wire Line
+	9950 4150 10100 4150
+Wire Wire Line
+	9500 4150 9500 4300
+Wire Wire Line
+	9500 4300 9100 4300
+Wire Wire Line
+	9950 4650 10100 4650
+Wire Wire Line
+	9500 4650 9500 4500
+Wire Wire Line
+	9500 4500 9100 4500
+Wire Wire Line
+	9100 4400 9650 4400
 $EndSCHEMATC
