File: hardware/boards/rev2/mixer.sch (KiCad schematic (older format))
At the start: 41 parts, among them U35 5400BL15B050E, U36 5400BL15B050E, U37 5400BL15B050E, U38 ADL5802

Commit message: reorganize schematic
Parts:
- removed F1, F2: Via-fmcw3-rescue, fmcw:RF_via, symbol fmcw-rescue:Via-fmcw3-rescue
- added JP10, JP9: miter_0.38_90deg, fmcw:uwmiter_0.38_0.17_90, symbol fmcw-rescue:miter_0.38_90deg
Connections:
- net LO_IN: now also JP9.1; no longer U35.1
- new net: JP10.2, U35.1
- new net: JP10.1, JP9.2
Other:
- note added: "300 (220) mA"
- note removed: "I_max: 300mA\nI_typ: 220mA"

Commit message: revert to kicad v5 for pcb gen
V6 contains a few bugs and a V6 board cannot be edited with V5.
Parts:
- removed JP1, JP10, JP15, JP16, JP8, JP9: miter_0.38_90deg, fmcw:uwmiter_0.38_0.17_90, symbol fmcw-rescue:miter_0.38_90deg
- added T3, T4, T5, T6, T7, T8: uwave, fmcw_v5:uwm_0.38_0.17_90, symbol fmcw:uwave
- C218, C219, C220, C221, C222, C223: footprint fmcw:RF_C_0201_0603Metric -> fmcw_v5:RF_C_0201_0603Metric
- JP17, JP2, JP4: footprint fmcw:balun_exit_inv -> fmcw_v5:balun_exit_inv
- JP18, JP3, JP5: footprint fmcw:balun_exit -> fmcw_v5:balun_exit
Connections:
- net LO_IN: now also U35.1, T3.1, T4.1
- net RF1: now also U37.1, T6.1
- net RF2: now also U36.1, T5.1, T7.1, T8.1
Changed lines of the file:
@@
-EESchema Schematic File Version 5
-EELAYER 33 0
+EESchema Schematic File Version 4
+EELAYER 30 0
 EELAYER END
 $Descr A4 11693 8268
 encoding utf-8
-Sheet 6 11
+Sheet 7 11
 Title "FMCW"
 Date ""
@@
 Comment3 ""
 Comment4 ""
-Comment5 ""
-Comment6 ""
-Comment7 ""
-Comment8 ""
-Comment9 ""
 $EndDescr
 Connection ~ 9950 4200
@@
 Connection ~ 7150 1150
 Connection ~ 6000 1150
-Wire Wire Line
-	1900 4200 2350 4200
-Wire Wire Line
-	2400 2350 2700 2350
-Wire Wire Line
-	2450 6450 2750 6450
-Wire Wire Line
-	2550 4000 2900 4000
-Wire Wire Line
-	2700 2150 2700 2350
-Wire Wire Line
-	3000 2150 2700 2150
-Wire Wire Line
-	3000 6250 2950 6250
-Wire Wire Line
-	3100 4200 3350 4200
-Wire Wire Line
-	3200 2350 3650 2350
-Wire Wire Line
-	3200 6450 3300 6450
+Connection ~ 2150 4200
+Connection ~ 2850 4200
+Connection ~ 2900 2350
+Connection ~ 2600 6450
+Connection ~ 3050 6450
+Connection ~ 3350 6450
+Wire Wire Line
+	1900 4200 2150 4200
+Wire Wire Line
+	2150 4200 2850 4200
+Wire Wire Line
+	2400 2350 2900 2350
+Wire Wire Line
+	2450 6450 2600 6450
+Wire Wire Line
+	2600 6450 3050 6450
+Wire Wire Line
+	2850 4200 3350 4200
+Wire Wire Line
+	2900 2350 3650 2350
+Wire Wire Line
+	3050 6450 3350 6450
 Wire Wire Line
 	3350 900  3500 900
 Wire Wire Line
+	3350 6450 3700 6450
+Wire Wire Line
 	3450 4700 3450 4800
 Wire Wire Line
@@
 	3500 1400 3500 1500
 Wire Wire Line
-	3500 6250 3700 6250
-Wire Wire Line
 	3550 2850 3750 2850
 Wire Wire Line
 	3550 2950 3550 2850
-Wire Wire Line
-	3700 6250 3700 6450
 Wire Wire Line
 	3750 4200 4100 4200
@@
 Text Notes 2300 1000 0    50   Italic 0
 300 (220) mA
+Text Label 4150 6450 0    50   ~ 0
+RF2a+
+Text Label 4150 6850 0    50   ~ 0
+RF2a-
 Text Label 4200 2350 0    50   ~ 0
 RF1a+
 Text Label 4200 2750 0    50   ~ 0
 RF1a-
-Text Label 4300 6450 0    50   ~ 0
-RF2a+
-Text Label 4300 6850 0    50   ~ 0
-RF2a-
 Text Label 4900 4150 0    50   ~ 0
 LOIa-
@@
 F 0 "JP17" H 4250 4000 50  0001 C CNN
 F 1 "balun_exit_inv" H 4250 4300 50  0001 C CNN
-F 2 "fmcw:balun_exit_inv" H 4250 4150 50  0001 C CNN
+F 2 "fmcw_v5:balun_exit_inv" H 4250 4150 50  0001 C CNN
 F 3 "" H 4250 4150 50  0001 C CNN
 	1    4250 4150
@@
 F 0 "JP18" H 4350 4450 50  0001 C CNN
 F 1 "balun_exit" H 4350 4750 50  0001 C CNN
-F 2 "fmcw:balun_exit" H 4350 4600 50  0001 C CNN
+F 2 "fmcw_v5:balun_exit" H 4350 4600 50  0001 C CNN
 F 3 "" H 4350 4600 50  0001 C CNN
 	1    4350 4600
@@
 F 0 "JP3" H 5050 6300 50  0001 C CNN
 F 1 "balun_exit" H 5050 6600 50  0001 C CNN
-F 2 "fmcw:balun_exit" H 5050 6450 50  0001 C CNN
+F 2 "fmcw_v5:balun_exit" H 5050 6450 50  0001 C CNN
 F 3 "" H 5050 6450 50  0001 C CNN
 	1    5050 6450
@@
 F 0 "JP2" H 5050 6550 50  0001 C CNN
 F 1 "balun_exit_inv" H 5050 6850 50  0001 C CNN
-F 2 "fmcw:balun_exit_inv" H 5050 6700 50  0001 C CNN
+F 2 "fmcw_v5:balun_exit_inv" H 5050 6700 50  0001 C CNN
 F 3 "" H 5050 6700 50  0001 C CNN
 	1    5050 6700
@@
 F 0 "JP5" H 5250 2200 50  0001 C CNN
 F 1 "balun_exit" H 5250 2500 50  0001 C CNN
-F 2 "fmcw:balun_exit" H 5250 2350 50  0001 C CNN
+F 2 "fmcw_v5:balun_exit" H 5250 2350 50  0001 C CNN
 F 3 "" H 5250 2350 50  0001 C CNN
 	1    5250 2350
@@
 F 0 "JP4" H 5250 2450 50  0001 C CNN
 F 1 "balun_exit_inv" H 5250 2750 50  0001 C CNN
-F 2 "fmcw:balun_exit_inv" H 5250 2600 50  0001 C CNN
+F 2 "fmcw_v5:balun_exit_inv" H 5250 2600 50  0001 C CNN
 F 3 "" H 5250 2600 50  0001 C CNN
 	1    5250 2600
 	1    0    0    -1
+$EndComp
+$Comp
+L fmcw:uwave T3
+U 1 1 5EAA2219
+P 2150 4350
+F 0 "T3" H 2022 4274 50  0000 R CNN
+F 1 "uwave" H 2022 4364 50  0000 R CNN
+F 2 "fmcw_v5:uwm_0.38_0.17_90" H 2150 4350 50  0001 C CNN
+F 3 "" H 2150 4350 50  0001 C CNN
+	1    2150 4350
+	-1   0    0    1
+$EndComp
+$Comp
+L fmcw:uwave T5
+U 1 1 5EA2D8AC
+P 2600 6600
+F 0 "T5" H 2472 6524 50  0000 R CNN
+F 1 "uwave" H 2472 6614 50  0000 R CNN
+F 2 "fmcw_v5:uwm_0.38_0.17_90" H 2600 6600 50  0001 C CNN
+F 3 "" H 2600 6600 50  0001 C CNN
+	1    2600 6600
+	-1   0    0    1
+$EndComp
+$Comp
+L fmcw:uwave T4
+U 1 1 5EAA704D
+P 2850 4350
+F 0 "T4" H 2722 4274 50  0000 R CNN
+F 1 "uwave" H 2722 4364 50  0000 R CNN
+F 2 "fmcw_v5:uwm_0.38_0.17_90" H 2850 4350 50  0001 C CNN
+F 3 "" H 2850 4350 50  0001 C CNN
+	1    2850 4350
+	-1   0    0    1
+$EndComp
+$Comp
+L fmcw:uwave T6
+U 1 1 5EA2CDA7
+P 2900 2500
+F 0 "T6" H 2772 2424 50  0000 R CNN
+F 1 "uwave" H 2772 2514 50  0000 R CNN
+F 2 "fmcw_v5:uwm_0.38_0.17_90" H 2900 2500 50  0001 C CNN
+F 3 "" H 2900 2500 50  0001 C CNN
+	1    2900 2500
+	-1   0    0    1
+$EndComp
+$Comp
+L fmcw:uwave T7
+U 1 1 5EA2E59B
+P 3050 6300
+F 0 "T7" H 2922 6224 50  0000 R CNN
+F 1 "uwave" H 2922 6314 50  0000 R CNN
+F 2 "fmcw_v5:uwm_0.38_0.17_90" H 3050 6300 50  0001 C CNN
+F 3 "" H 3050 6300 50  0001 C CNN
+	1    3050 6300
+	1    0    0    -1
+$EndComp
+$Comp
+L fmcw:uwave T8
+U 1 1 5EA3B500
+P 3350 6600
+F 0 "T8" H 3222 6524 50  0000 R CNN
+F 1 "uwave" H 3222 6614 50  0000 R CNN
+F 2 "fmcw_v5:uwm_0.38_0.17_90" H 3350 6600 50  0001 C CNN
+F 3 "" H 3350 6600 50  0001 C CNN
+	1    3350 6600
+	-1   0    0    1
 $EndComp
 $Comp
@@
 F 0 "C220" V 5148 4200 50  0000 C CNN
 F 1 "10p" V 5239 4200 50  0000 C CNN
-F 2 "fmcw:RF_C_0201_0603Metric" H 5438 4050 30  0001 C CNN
+F 2 "fmcw_v5:RF_C_0201_0603Metric" H 5438 4050 30  0001 C CNN
 F 3 "" H 5400 4200 60  0000 C CNN
 F 4 "GJM0335C1E100GB01D" H 1850 250 50  0001 C CNN "MFN"
@@
 F 0 "C221" V 5560 4400 50  0000 C CNN
 F 1 "10p" V 5651 4400 50  0000 C CNN
-F 2 "fmcw:RF_C_0201_0603Metric" H 5438 4250 30  0001 C CNN
+F 2 "fmcw_v5:RF_C_0201_0603Metric" H 5438 4250 30  0001 C CNN
 F 3 "" H 5400 4400 60  0000 C CNN
 F 4 "GJM0335C1E100GB01D" H 1850 250 50  0001 C CNN "MFN"
@@
 F 0 "C222" V 5648 6450 50  0000 C CNN
 F 1 "10p" V 5739 6450 50  0000 C CNN
-F 2 "fmcw:RF_C_0201_0603Metric" H 5938 6300 30  0001 C CNN
+F 2 "fmcw_v5:RF_C_0201_0603Metric" H 5938 6300 30  0001 C CNN
 F 3 "" H 5900 6450 60  0000 C CNN
 F 4 "GJM0335C1E100GB01D" H 2350 550 50  0001 C CNN "MFN"
@@
 F 0 "C223" V 6060 6650 50  0000 C CNN
 F 1 "10p" V 6151 6650 50  0000 C CNN
-F 2 "fmcw:RF_C_0201_0603Metric" H 5938 6500 30  0001 C CNN
+F 2 "fmcw_v5:RF_C_0201_0603Metric" H 5938 6500 30  0001 C CNN
 F 3 "" H 5900 6650 60  0000 C CNN
 F 4 "GJM0335C1E100GB01D" H 2350 550 50  0001 C CNN "MFN"
@@
 F 0 "C218" V 5900 2550 50  0000 C CNN
 F 1 "10p" V 5789 2350 50  0000 C CNN
-F 2 "fmcw:RF_C_0201_0603Metric" H 5988 2200 30  0001 C CNN
+F 2 "fmcw_v5:RF_C_0201_0603Metric" H 5988 2200 30  0001 C CNN
 F 3 "" H 5950 2350 60  0000 C CNN
 F 4 "GJM0335C1E100GB01D" H 2400 -2550 50  0001 C CNN "MFN"
@@
 F 0 "C219" V 6110 2550 50  0000 C CNN
 F 1 "10p" V 6201 2550 50  0000 C CNN
-F 2 "fmcw:RF_C_0201_0603Metric" H 5988 2400 30  0001 C CNN
+F 2 "fmcw_v5:RF_C_0201_0603Metric" H 5988 2400 30  0001 C CNN
 F 3 "" H 5950 2550 60  0000 C CNN
 F 4 "GJM0335C1E100GB01D" H 2400 -2550 50  0001 C CNN "MFN"
@@
 $EndComp
 $Comp
-L fmcw-rescue:miter_0.38_90deg JP9
-U 1 1 5E9D4C6A
-P 2500 4150
-F 0 "JP9" H 2550 4100 50  0001 C CNN
-F 1 "miter_0.38_90deg" H 2528 4333 50  0000 C CNN
-F 2 "fmcw:uwmiter_0.38_0.17_90" H 2500 4100 50  0001 C CNN
-F 3 "" H 2500 4100 50  0001 C CNN
-	1    2500 4150
-	-1   0    0    1
-$EndComp
-$Comp
-L fmcw-rescue:miter_0.38_90deg JP8
-U 1 1 5EA9F129
-P 2800 6300
-F 0 "JP8" H 2828 6483 50  0000 C CNN
-F 1 "miter_0.38_90deg" H 2828 6484 50  0001 C CNN
-F 2 "fmcw:uwmiter_0.38_0.17_90" H 2800 6250 50  0001 C CNN
-F 3 "" H 2800 6250 50  0001 C CNN
-	1    2800 6300
-	1    0    0    -1
-$EndComp
-$Comp
-L fmcw-rescue:miter_0.38_90deg JP10
-U 1 1 5E9F563F
-P 2950 4150
-F 0 "JP10" H 3000 4100 50  0001 C CNN
-F 1 "miter_0.38_90deg" V 3200 3850 50  0000 L CNN
-F 2 "fmcw:uwmiter_0.38_0.17_90" H 2950 4100 50  0001 C CNN
-F 3 "" H 2950 4100 50  0001 C CNN
-	1    2950 4150
-	0    -1   -1   0
-$EndComp
-$Comp
-L fmcw-rescue:miter_0.38_90deg JP1
-U 1 1 5E94277D
-P 3050 2300
-F 0 "JP1" V 3100 2150 50  0000 L CNN
-F 1 "miter_0.38_90deg" V 2850 2150 50  0000 L CNN
-F 2 "fmcw:uwmiter_0.38_0.17_90" H 3050 2250 50  0001 C CNN
-F 3 "" H 3050 2250 50  0001 C CNN
-	1    3050 2300
-	0    -1   -1   0
-$EndComp
-$Comp
-L fmcw-rescue:miter_0.38_90deg JP15
-U 1 1 5EAE170F
-P 3050 6400
-F 0 "JP15" V 2800 6372 50  0000 C CNN
-F 1 "miter_0.38_90deg" H 3078 6584 50  0001 C CNN
-F 2 "fmcw:uwmiter_0.38_0.17_90" H 3050 6350 50  0001 C CNN
-F 3 "" H 3050 6350 50  0001 C CNN
-	1    3050 6400
-	0    -1   -1   0
-$EndComp
-$Comp
-L fmcw-rescue:miter_0.38_90deg JP16
-U 1 1 5EAE6CC4
-P 3450 6400
-F 0 "JP16" H 3478 6650 50  0000 C CNN
-F 1 "miter_0.38_90deg" H 3478 6584 50  0001 C CNN
-F 2 "fmcw:uwmiter_0.38_0.17_90" H 3450 6350 50  0001 C CNN
-F 3 "" H 3450 6350 50  0001 C CNN
-	1    3450 6400
-	-1   0    0    1
-$EndComp
-$Comp
 L Transformer:5400BL15B050 U35
 U 1 1 5D0263FC
@@
 U 1 1 5D050232
 P 3900 6650
-F 0 "U36" H 3900 7075 50  0000 C CNN
-F 1 "5400BL15B050E" H 3900 6984 50  0000 C CNN
+F 0 "U36" H 3900 7070 50  0000 C CNN
+F 1 "5400BL15B050E" H 3900 6979 50  0000 C CNN
 F 2 "RF_Converter:Balun_Johanson_5400BL15B050E" H 3900 6400 50  0001 C CNN
 F 3 "" H 3900 6400 50  0001 C CNN

Commit message: finish placement and routing
Parts:
- removed JP17, JP2, JP4: balun_exit_inv, fmcw_v5:balun_exit_inv, symbol fmcw-rescue:balun_exit_inv
- removed JP18, JP3, JP5: balun_exit, fmcw_v5:balun_exit, symbol fmcw-rescue:balun_exit
- added T10, T11, T12: uwave, fmcw_v5:balun_exit_inv, symbol fmcw:uwave
- added T13, T14, T9: uwave, fmcw_v5:balun_exit, symbol fmcw:uwave
Connections:
- net LOIa+: now also U35.4, T9.1
- net LOIa-: now also U35.3, T10.1
- net RF1a+: now also C219.2, T11.1
- net RF1a-: now also C218.2, T13.1
- net RF2a+: now also C223.2, T12.1
- net RF2a-: now also C222.2, T14.1
Changed lines of the file:
@@
 	3550 2950 3550 2850
 Wire Wire Line
-	3750 4200 4100 4200
-Wire Wire Line
-	3750 4600 4200 4600
-Wire Wire Line
 	3800 7050 3800 6950
 Wire Wire Line
@@
 	4350 2550 4350 2350
 Wire Wire Line
-	4350 2550 5100 2550
+	4350 2550 4850 2550
 Wire Wire Line
 	4350 6650 4350 6450
 Wire Wire Line
-	4350 6650 4900 6650
-Wire Wire Line
-	4400 4150 5050 4150
+	4350 6650 4750 6650
 Wire Wire Line
 	4450 2350 4450 2750
 Wire Wire Line
-	4450 2350 5100 2350
+	4450 2350 4900 2350
 Wire Wire Line
 	4450 6450 4450 6850
 Wire Wire Line
-	4450 6450 4900 6450
-Wire Wire Line
 	4450 6850 4100 6850
 Wire Wire Line
-	4500 4650 5150 4650
-Wire Wire Line
-	4900 6650 4900 6750
-Wire Wire Line
 	5000 1150 5350 1150
 Wire Wire Line
-	5050 4150 5050 4400
-Wire Wire Line
 	5050 4400 5250 4400
 Wire Wire Line
-	5100 2550 5100 2650
-Wire Wire Line
-	5150 4200 5150 4650
-Wire Wire Line
-	5200 6400 5200 6500
-Wire Wire Line
-	5200 6400 5350 6400
-Wire Wire Line
-	5200 6700 5350 6700
+	5150 4200 5150 4600
 Wire Wire Line
 	5250 4200 5150 4200
 Wire Wire Line
 	5350 1150 5700 1150
-Wire Wire Line
-	5350 6400 5350 6450
-Wire Wire Line
-	5350 6450 5750 6450
-Wire Wire Line
-	5350 6650 5750 6650
-Wire Wire Line
-	5350 6700 5350 6650
-Wire Wire Line
-	5400 2400 5550 2400
-Wire Wire Line
-	5400 2600 5550 2600
-Wire Wire Line
-	5550 2350 5800 2350
-Wire Wire Line
-	5550 2400 5550 2350
-Wire Wire Line
-	5550 2550 5800 2550
-Wire Wire Line
-	5550 2600 5550 2550
 Wire Wire Line
 	5700 900  5700 1150
@@
 Text Label 4200 2750 0    50   ~ 0
 RF1a-
-Text Label 4900 4150 0    50   ~ 0
+Text Label 4900 4200 0    50   ~ 0
 LOIa-
-Text Label 4900 4650 0    50   ~ 0
+Text Label 4900 4600 0    50   ~ 0
 LOIa+
 Text Label 6200 4050 0    50   ~ 0
@@
 $EndComp
 $Comp
-L fmcw-rescue:balun_exit_inv JP17
-U 1 1 5E845684
-P 4250 4150
-F 0 "JP17" H 4250 4000 50  0001 C CNN
-F 1 "balun_exit_inv" H 4250 4300 50  0001 C CNN
-F 2 "fmcw_v5:balun_exit_inv" H 4250 4150 50  0001 C CNN
-F 3 "" H 4250 4150 50  0001 C CNN
-	1    4250 4150
-	1    0    0    -1
-$EndComp
-$Comp
-L fmcw-rescue:balun_exit JP18
-U 1 1 5E8444EB
-P 4350 4600
-F 0 "JP18" H 4350 4450 50  0001 C CNN
-F 1 "balun_exit" H 4350 4750 50  0001 C CNN
-F 2 "fmcw_v5:balun_exit" H 4350 4600 50  0001 C CNN
-F 3 "" H 4350 4600 50  0001 C CNN
-	1    4350 4600
-	1    0    0    -1
-$EndComp
-$Comp
-L fmcw-rescue:balun_exit JP3
-U 1 1 5E9C956A
-P 5050 6450
-F 0 "JP3" H 5050 6300 50  0001 C CNN
-F 1 "balun_exit" H 5050 6600 50  0001 C CNN
-F 2 "fmcw_v5:balun_exit" H 5050 6450 50  0001 C CNN
-F 3 "" H 5050 6450 50  0001 C CNN
-	1    5050 6450
-	1    0    0    -1
-$EndComp
-$Comp
-L fmcw-rescue:balun_exit_inv JP2
-U 1 1 5E9C9398
-P 5050 6700
-F 0 "JP2" H 5050 6550 50  0001 C CNN
-F 1 "balun_exit_inv" H 5050 6850 50  0001 C CNN
-F 2 "fmcw_v5:balun_exit_inv" H 5050 6700 50  0001 C CNN
-F 3 "" H 5050 6700 50  0001 C CNN
-	1    5050 6700
-	1    0    0    -1
-$EndComp
-$Comp
-L fmcw-rescue:balun_exit JP5
-U 1 1 5E9C2CE4
-P 5250 2350
-F 0 "JP5" H 5250 2200 50  0001 C CNN
-F 1 "balun_exit" H 5250 2500 50  0001 C CNN
-F 2 "fmcw_v5:balun_exit" H 5250 2350 50  0001 C CNN
-F 3 "" H 5250 2350 50  0001 C CNN
-	1    5250 2350
-	1    0    0    -1
-$EndComp
-$Comp
-L fmcw-rescue:balun_exit_inv JP4
-U 1 1 5E9BE4F9
-P 5250 2600
-F 0 "JP4" H 5250 2450 50  0001 C CNN
-F 1 "balun_exit_inv" H 5250 2750 50  0001 C CNN
-F 2 "fmcw_v5:balun_exit_inv" H 5250 2600 50  0001 C CNN
-F 3 "" H 5250 2600 50  0001 C CNN
-	1    5250 2600
-	1    0    0    -1
-$EndComp
-$Comp
 L fmcw:uwave T3
 U 1 1 5EAA2219
@@
 	1    0    0    -1
 $EndComp
+$Comp
+L fmcw:uwave T9
+U 1 1 5EB3AE17
+P 4300 4750
+F 0 "T9" H 4172 4674 50  0000 R CNN
+F 1 "uwave" H 4172 4764 50  0000 R CNN
+F 2 "fmcw_v5:balun_exit" H 4300 4750 50  0001 C CNN
+F 3 "" H 4300 4750 50  0001 C CNN
+	1    4300 4750
+	-1   0    0    1
+$EndComp
+Wire Wire Line
+	3750 4600 4300 4600
+Wire Wire Line
+	4300 4600 5150 4600
+Connection ~ 4300 4600
+$Comp
+L fmcw:uwave T10
+U 1 1 5EB4F53D
+P 4250 4050
+F 0 "T10" H 4378 4063 50  0000 L CNN
+F 1 "uwave" H 4378 3972 50  0000 L CNN
+F 2 "fmcw_v5:balun_exit_inv" H 4250 4050 50  0001 C CNN
+F 3 "" H 4250 4050 50  0001 C CNN
+	1    4250 4050
+	1    0    0    -1
+$EndComp
+Wire Wire Line
+	3750 4200 4250 4200
+Wire Wire Line
+	4250 4200 5050 4200
+Connection ~ 4250 4200
+Wire Wire Line
+	5050 4200 5050 4400
+$Comp
+L fmcw:uwave T11
+U 1 1 5EB59BEA
+P 4850 2700
+F 0 "T11" H 4850 2873 50  0000 C CNN
+F 1 "uwave" H 4850 2964 50  0000 C CNN
+F 2 "fmcw_v5:balun_exit_inv" H 4850 2700 50  0001 C CNN
+F 3 "" H 4850 2700 50  0001 C CNN
+	1    4850 2700
+	-1   0    0    1
+$EndComp
+Connection ~ 4850 2550
+Wire Wire Line
+	4850 2550 5800 2550
+$Comp
+L fmcw:uwave T13
+U 1 1 5EB63605
+P 4900 2200
+F 0 "T13" H 4772 2124 50  0000 R CNN
+F 1 "uwave" H 4772 2214 50  0000 R CNN
+F 2 "fmcw_v5:balun_exit" H 4900 2200 50  0001 C CNN
+F 3 "" H 4900 2200 50  0001 C CNN
+	1    4900 2200
+	1    0    0    -1
+$EndComp
+Connection ~ 4900 2350
+Wire Wire Line
+	4900 2350 5800 2350
+$Comp
+L fmcw:uwave T14
+U 1 1 5EB68520
+P 5100 6300
+F 0 "T14" H 4972 6224 50  0000 R CNN
+F 1 "uwave" H 4972 6314 50  0000 R CNN
+F 2 "fmcw_v5:balun_exit" H 5100 6300 50  0001 C CNN
+F 3 "" H 5100 6300 50  0001 C CNN
+	1    5100 6300
+	1    0    0    -1
+$EndComp
+$Comp
+L fmcw:uwave T12
+U 1 1 5EB6BD86
+P 4750 6800
+F 0 "T12" H 4750 6973 50  0000 C CNN
+F 1 "uwave" H 4750 7064 50  0000 C CNN
+F 2 "fmcw_v5:balun_exit_inv" H 4750 6800 50  0001 C CNN
+F 3 "" H 4750 6800 50  0001 C CNN
+	1    4750 6800
+	-1   0    0    1
+$EndComp
+Connection ~ 4750 6650
+Wire Wire Line
+	4750 6650 5750 6650
+Connection ~ 5100 6450
+Wire Wire Line
+	5100 6450 5750 6450
+Wire Wire Line
+	4450 6450 5100 6450
 $EndSCHEMATC
