File: hardware/boards/rev2/tx.sch (KiCad schematic (older format))
At the start: 64 parts, among them J3 SMA, Q2 RE1C002UN, U12 ADF4158, U13 TLV172DCK, U14 PAT1220-C-3DB, U15 HMC431LP4, U16 PD4859J5050S2HF, U17 PAT1220-C-5DB, U18 SE5004L, U20 PAT1220-C-6DB, U21 LMV321

Commit message: reorganize schematic
Parts:
- removed C128, C133, C134: DNP, Capacitor_SMD:C_0402_1005Metric, symbol Device:C
- removed C136: 100n, Capacitor_SMD:C_0402_1005Metric, symbol Device:C
- removed C137: DNP, Capacitor_SMD:C_0603_1608Metric, symbol Device:C
- U18: symbol RF:SE5004L -> fmcw:SE5004L
Connections:
- net labels added: 5V_PA, 5V_SYNTH
- wire segments 239 -> 222
- no-connect marks 1 -> 2
Other:
- note added: "10 mA"
- note added: "3 mA"
- note added: "32 (23) mA"
- note added: "5 mA"
- note added: "800 (300) mA"
- note removed: "10V current: 1mA\n3.3V current: 600mA\n5V current: 1mA"
- note removed: "35 mA"
- note removed: "I_max: 800mA\nI_q: 300mA"
- moved on the sheet: C252

Commit message: revert to kicad v5 for pcb gen
V6 contains a few bugs and a V6 board cannot be edited with V5.
Parts:
- removed JP6, JP7: miter_0.38_90deg, fmcw:uwmiter_0.38_0.17_90, symbol fmcw-rescue:miter_0.38_90deg
- added T1, T2: uwave, fmcw_v5:uwm_0.38_0.17_90, symbol fmcw:uwave
- C112, C251, C252, C267: footprint fmcw:RF_C_0201_0603Metric -> fmcw_v5:RF_C_0201_0603Metric
- J3: footprint fmcw:BU-1420701851_SMA -> fmcw_v5:SMA_901-10512
- R47: footprint fmcw:R_0603b -> fmcw_v5:R_0603b
- U15: value HMC431LP4 -> HMC431; symbol RF:HMC431 -> fmcw:HMC431
- U18: footprint fmcw:Skyworks_SE5004L -> fmcw_v5:Skyworks_SE5004L
- Z1: footprint fmcw:coupler_20db -> fmcw_v5:coupler_20db
Connections:
- net GND: now also U15.1 (NC), U15.10 (NC), U15.11 (NC), U15.12 (NC), U15.13 (NC), U15.14 (NC), U15.17 (NC), U15.18 (NC), U15.19 (NC), U15.2 (NC), U15.21 (NC), U15.23 (NC), U15.24 (NC), U15.3 (NC), U15.4 (NC), U15.5 (NC), U15.6 (NC), U15.7 (NC), U15.8 (NC), U15.9 (NC)
- net TX_COUPLED: now also U20.1; no longer U20.2
- net at Z1.3: now also U20.2; no longer U20.1
- net at R47.2, U16.6 (Output2): now also U14.2, T1.1, T2.1
Changed lines of the file:
@@
-EESchema Schematic File Version 5
-EELAYER 33 0
+EESchema Schematic File Version 4
+EELAYER 30 0
 EELAYER END
 $Descr A3 16535 11693
 encoding utf-8
-Sheet 6 11
+Sheet 11 11
 Title "FMCW"
 Date ""
@@
 Comment3 ""
 Comment4 ""
-Comment5 ""
-Comment6 ""
-Comment7 ""
-Comment8 ""
-Comment9 ""
 $EndDescr
 Connection ~ 2200 5250
@@
 Connection ~ 9950 5800
 Connection ~ 9950 6200
-Connection ~ 8150 5250
 Connection ~ 8150 5050
 Connection ~ 6200 5550
@@
 Connection ~ 11900 2900
 Connection ~ 11900 2650
+Connection ~ 8150 5250
+Connection ~ 8150 6400
+Connection ~ 9300 7450
+Connection ~ 9950 7150
 NoConn ~ 2900 5800
 NoConn ~ 12500 4800
@@
 	7600 4900 8050 4900
 Wire Wire Line
+	7750 6100 7750 6400
+Wire Wire Line
+	7750 6400 8150 6400
+Wire Wire Line
 	7800 7850 7800 7900
 Wire Wire Line
@@
 	8150 5250 8150 5700
 Wire Wire Line
-	8150 6350 8150 6300
+	8150 6400 8150 6300
+Wire Wire Line
+	8150 6400 8150 6500
 Wire Wire Line
 	8200 5250 8150 5250
 Wire Wire Line
-	8200 7450 9450 7450
+	8200 7450 9300 7450
 Wire Wire Line
 	8250 3550 8250 3600
@@
 	9150 4450 9150 4200
 Wire Wire Line
+	9300 7450 9300 7550
+Wire Wire Line
+	9300 7450 9950 7450
+Wire Wire Line
 	9400 6350 9400 6300
 Wire Wire Line
@@
 	9450 4400 9450 4900
 Wire Wire Line
-	9450 7300 9450 7450
-Wire Wire Line
 	9500 4450 9150 4450
 Wire Wire Line
 	9550 3550 9450 3550
 Wire Wire Line
-	9750 6950 9750 7100
-Wire Wire Line
-	9750 7100 9650 7100
-Wire Wire Line
 	9800 5900 9850 5900
 Wire Wire Line
@@
 	9950 6150 9950 6200
 Wire Wire Line
-	9950 6200 9950 6750
+	9950 6200 9950 7150
+Wire Wire Line
+	9950 7150 9950 7450
 Wire Wire Line
 	10050 4100 10050 4300
@@
 L power:GND #PWR0117
 U 1 1 54FADCB5
-P 8150 6350
-F 0 "#PWR0117" H 8150 6350 30  0001 C CNN
-F 1 "GND" H 8150 6280 30  0001 C CNN
-F 2 "" H 8150 6350 60  0000 C CNN
-F 3 "" H 8150 6350 60  0000 C CNN
-	1    8150 6350
+P 8150 6500
+F 0 "#PWR0117" H 8150 6500 30  0001 C CNN
+F 1 "GND" H 8150 6430 30  0001 C CNN
+F 2 "" H 8150 6500 60  0000 C CNN
+F 3 "" H 8150 6500 60  0000 C CNN
+	1    8150 6500
 	1    0    0    -1
 $EndComp
@@
 F 0 "R47" H 10020 6046 50  0000 L CNN
 F 1 "100" H 10020 5955 50  0000 L CNN
-F 2 "fmcw:R_0603b" V 9880 6000 50  0001 C CNN
+F 2 "fmcw_v5:R_0603b" V 9880 6000 50  0001 C CNN
 F 3 "~" H 9950 6000 50  0001 C CNN
 F 4 "" H 9950 6000 50  0001 C CNN "MFN"
@@
 $EndComp
 $Comp
+L fmcw:uwave T1
+U 1 1 5EAFC5E6
+P 9300 7700
+F 0 "T1" H 9172 7624 50  0000 R CNN
+F 1 "uwave" H 9172 7714 50  0000 R CNN
+F 2 "fmcw_v5:uwm_0.38_0.17_90" H 9300 7700 50  0001 C CNN
+F 3 "" H 9300 7700 50  0001 C CNN
+	1    9300 7700
+	-1   0    0    1
+$EndComp
+$Comp
+L fmcw:uwave T2
+U 1 1 5EB0CF7E
+P 10100 7150
+F 0 "T2" V 10055 7278 50  0000 L CNN
+F 1 "uwave" V 10145 7278 50  0000 L CNN
+F 2 "fmcw_v5:uwm_0.38_0.17_90" H 10100 7150 50  0001 C CNN
+F 3 "" H 10100 7150 50  0001 C CNN
+	1    10100 7150
+	0    1    1    0
+$EndComp
+$Comp
 L Device:C C102
 U 1 1 54FAB845
@@
 F 0 "C112" V 4021 7450 40  0000 C CNN
 F 1 "10p" V 4097 7450 40  0000 C CNN
-F 2 "fmcw:RF_C_0201_0603Metric" H 4288 7300 30  0001 C CNN
+F 2 "fmcw_v5:RF_C_0201_0603Metric" H 4288 7300 30  0001 C CNN
 F 3 "" H 4250 7450 60  0000 C CNN
 F 4 "GJM0335C1E100GB01D" H -950 100 50  0001 C CNN "MFN"
@@
 F 0 "C251" V 10950 5100 50  0000 C CNN
 F 1 "10p" V 11250 5100 50  0000 C CNN
-F 2 "fmcw:RF_C_0201_0603Metric" H 11138 4950 50  0001 C CNN
+F 2 "fmcw_v5:RF_C_0201_0603Metric" H 11138 4950 50  0001 C CNN
 F 3 "~" H 11100 5100 50  0001 C CNN
 F 4 "GJM0335C1E100GB01D" H -600 600 50  0001 C CNN "MFN"
@@
 F 0 "C252" V 12850 5100 50  0000 C CNN
 F 1 "10p" V 12950 5100 50  0000 C CNN
-F 2 "fmcw:RF_C_0201_0603Metric" H 13138 4950 50  0001 C CNN
+F 2 "fmcw_v5:RF_C_0201_0603Metric" H 13138 4950 50  0001 C CNN
 F 3 "~" H 13100 5100 50  0001 C CNN
 F 4 "GJM0335C1E100GB01D" H 1750 500 50  0001 C CNN "MFN"
@@
 F 0 "C267" H 13235 5304 50  0000 R CNN
 F 1 "0.3p" H 13235 5395 50  0000 R CNN
-F 2 "fmcw:RF_C_0201_0603Metric" H 13388 5200 50  0001 C CNN
+F 2 "fmcw_v5:RF_C_0201_0603Metric" H 13388 5200 50  0001 C CNN
 F 3 "~" H 13350 5350 50  0001 C CNN
 F 4 "GJM0335C1ER30BB01D" H 2000 750 50  0001 C CNN "MFN"
@@
 $EndComp
 $Comp
-L fmcw-rescue:miter_0.38_90deg JP6
-U 1 1 5EB543D2
-P 9500 7150
-F 0 "JP6" H 9550 7100 50  0001 C CNN
-F 1 "miter_0.38_90deg" H 9366 7122 50  0000 R CNN
-F 2 "fmcw:uwmiter_0.38_0.17_90" H 9500 7100 50  0001 C CNN
-F 3 "" H 9500 7100 50  0001 C CNN
-	1    9500 7150
-	1    0    0    -1
-$EndComp
-$Comp
-L fmcw-rescue:miter_0.38_90deg JP7
-U 1 1 5EB539C0
-P 9800 6800
-F 0 "JP7" H 9850 6750 50  0001 C CNN
-F 1 "miter_0.38_90deg" H 9666 6772 50  0000 R CNN
-F 2 "fmcw:uwmiter_0.38_0.17_90" H 9800 6750 50  0001 C CNN
-F 3 "" H 9800 6750 50  0001 C CNN
-	1    9800 6800
-	1    0    0    -1
-$EndComp
-$Comp
 L Connector:Conn_Coaxial J3
 U 1 1 54FAB57F
@@
 F 0 "J3" H 15550 5083 60  0000 L CNN
 F 1 "SMA" H 15550 4977 60  0000 L CNN
-F 2 "fmcw:BU-1420701851_SMA" H 15450 5100 60  0001 C CNN
+F 2 "fmcw_v5:SMA_901-10512" H 15450 5100 60  0001 C CNN
 F 3 "" H 15450 5100 60  0000 C CNN
 F 4 "BU-1420701851" H -300 100 50  0001 C CNN "MFN"
@@
 F 0 "Z1" H 14450 5753 60  0000 C CNN
 F 1 "BRANCHLINE-fmcw3-rescue" H 14450 5647 60  0000 C CNN
-F 2 "fmcw:coupler_20db" H 14450 5541 60  0000 C CNN
+F 2 "fmcw_v5:coupler_20db" H 14450 5541 60  0000 C CNN
 F 3 "" H 14500 5100 60  0000 C CNN
 	1    14450 5250
@@
 F 4 "PAT1220-C-6DB-T5" H -400 350 50  0001 C CNN "MFN"
 	1    13800 6200
-	0    1    1    0
-$EndComp
-$Comp
-L RF:HMC431 U?
+	0    1    -1   0
+$EndComp
+$Comp
+L fmcw:HMC431 U?
 U 1 1 54FAAD5A
 P 8150 6000
 AR Path="/54FAAD5A" Ref="U?"  Part="1"
 AR Path="/59396B94/54FAAD5A" Ref="U15"  Part="1"
-F 0 "U15" H 8300 6350 60  0000 C CNN
-F 1 "HMC431LP4" H 8450 6250 60  0000 C CNN
+F 0 "U15" H 7900 6350 60  0000 C CNN
+F 1 "HMC431" H 8400 6350 60  0000 C CNN
 F 2 "Package_DFN_QFN:QFN-24-1EP_4x4mm_P0.5mm_EP2.8x2.8mm_ThermalVias" H 8150 6000 60  0001 C CNN
 F 3 "" H 8150 6000 60  0001 C CNN
@@
 F 0 "U18" H 12450 5250 50  0000 L CNN
 F 1 "SE5004L" H 11750 4800 50  0000 L CNN
-F 2 "fmcw:Skyworks_SE5004L" H 11800 4700 50  0001 C CNN
+F 2 "fmcw_v5:Skyworks_SE5004L" H 11800 4700 50  0001 C CNN
 F 3 "http://www.skyworksinc.com/uploads/documents/SE5004L_202393B.pdf" H 11900 4800 50  0001 C CNN
 F 4 "SE5004L-R" H -700 100 50  0001 C CNN "MFN"

Commit message: finish placement and routing
Parts:
- U15: symbol fmcw:HMC431 -> RF:HMC431
Changed lines of the file:
@@
 $EndComp
 $Comp
-L fmcw:HMC431 U?
+L RF:HMC431 U?
 U 1 1 54FAAD5A
 P 8150 6000

Commit message: switch ftclk to MRCC pin and place silkscreen
Parts:
- J3: MFN BU-1420701851 -> 901-10512-3
Changed lines of the file:
@@
 F 2 "fmcw_v5:SMA_901-10512" H 15450 5100 60  0001 C CNN
 F 3 "" H 15450 5100 60  0000 C CNN
-F 4 "BU-1420701851" H -300 100 50  0001 C CNN "MFN"
+F 4 "901-10512-3" H -300 100 50  0001 C CNN "MFN"
 	1    15450 5100
 	1    0    0    -1
